Commit message: fix : urdf fix

File: openarm_v1_bimanual_description/urdf/openarm_v1_bimanual.urdf (robot description, URDF)
Before this commit: robot openarm_v1_bimanual, 40 links, 39 joints
Links:
- link left_oparm_link8_1: mass 0.5019344947868502 -> 1.0519344947868502
- link right_oparm_link8_1: mass 0.5319344947868502 -> 1.0519344947868502

Commit message: add: dae stl

File: openarm_v1_bimanual_description/urdf/openarm_v1_bimanual.urdf (robot description, URDF)
Before this commit: robot openarm_v1_bimanual, 40 links, 39 joints
Links:
- link pedestal_v1_link: mass 13.892221893766356 -> None
