Commit message: fix: hand position

File: openarm_description/urdf/body/openarm_body.xacro (robot description, xacro)
@@ -29,15 +29,3 @@
     kinematics_link="${kinematics_link}" />
     </xacro:macro>
-    <!-- for bimanual right side-->
-    <!-- <joint name="${body_type}_body_to_right_${arm_type}_joint" type="fixed">
-      <origin xyz="0.3 -0.2 0.4" rpy="0 0 0" />
-      <parent link="body_link0" />
-      <child link="right_${arm_type}_link0" />
-    </joint> -->
-    <!-- for bimanual left side-->
-    <!-- <joint name="${body_type}_body_to_left_${arm_type}_joint" type="fixed">
-      <origin xyz="0.3 0.2 0.4" rpy="0 0 0" />
-      <parent link="body_link0" />
-      <child link="left_${arm_type}_link0" />
-    </joint> -->
 </robot>

File: openarm_description/urdf/ee/openarm_hand.xacro (robot description, xacro)
@@ -14,5 +14,6 @@
       </joint>
     </xacro:unless>
-    <xacro:ee_link_with_sc name="hand" gazebo="${gazebo}" />
+    <!-- <xacro:ee_link_with_sc name="hand" gazebo="${gazebo}" prefix="${ee_prefix}" ee_kinematics_link="${ee_kinematics_link}"/> -->
+    <link name="${ee_prefix}hand"/>
     <!-- Define the hand_tcp frame -->
     <link name="${ee_prefix}hand_tcp" />
@@ -24,8 +25,15 @@
     <link name="${ee_prefix}leftfinger">
       <visual name="${ee_prefix}leftfinger_visual">
+        <xacro:openarm-ee-kinematics-link config="${ee_kinematics_link}" name="leftfinger" />
         <geometry>
           <mesh filename="package://${description_pkg}/meshes/ee/${ee_type}/visual/finger.dae" scale="0.001 0.001 0.001"/>
         </geometry>
       </visual>
+      <collision name="${ee_prefix}leftfinger_collision">
+        <xacro:openarm-ee-kinematics-link config="${ee_kinematics_link}" name="leftfinger" />
+        <geometry>
+          <mesh filename="package://${description_pkg}/meshes/ee/${ee_type}/collision/finger.stl" scale="0.001 0.001 0.001" />
+        </geometry>
+      </collision>
       <xacro:if value="${gazebo}">
         <xacro:ee-inertials name="leftfinger" />
@@ -34,9 +42,15 @@
     <link name="${ee_prefix}rightfinger">
       <visual name="${ee_prefix}rightfinger_visual">
-        <origin xyz="0 0 0" rpy="0 0 ${pi}" />
+        <xacro:openarm-ee-kinematics-link config="${ee_kinematics_link}" name="rightfinger" />
         <geometry>
-          <mesh filename="package://${description_pkg}/meshes/ee/${ee_type}/visual/finger.dae" scale="0.001 0.001 0.001"/>
+          <mesh filename="package://${description_pkg}/meshes/ee/${ee_type}/visual/finger.dae" scale="0.001 -0.001 0.001"/>
         </geometry>
       </visual>
+      <collision name="${ee_prefix}rightfinger_collision">
+        <xacro:openarm-ee-kinematics-link config="${ee_kinematics_link}" name="leftfinger" />
+        <geometry>
+          <mesh filename="package://${description_pkg}/meshes/ee/${ee_type}/collision/finger.stl" scale="0.001 -0.001 0.001" />
+        </geometry>
+      </collision>
       <xacro:if value="${gazebo}">
         <xacro:ee-inertials name="rightfinger" />
@@ -47,13 +61,13 @@
       <child link="${ee_prefix}leftfinger" />
       <origin xyz="0 0 0" rpy="0 0 0" />
-      <axis xyz="0 1 0" />
-      <limit effort="100" lower="0.0" upper="0.04" velocity="0.2" />
+      <axis xyz="0 -1 0" />
+      <limit effort="100" lower="0.0" upper="0.044" velocity="0.2" />
     </joint>
     <joint name="${ee_prefix}finger_joint2" type="prismatic">
       <parent link="${ee_prefix}hand" />
       <child link="${ee_prefix}rightfinger" />
-      <origin xyz="0 0 0.0" rpy="0 0 0" />
-      <axis xyz="0 -1 0" />
-      <limit effort="100" lower="0.0" upper="0.04" velocity="0.2" />
+      <origin xyz="0 0 0" rpy="0 0 0" />
+      <axis xyz="0 1 0" />
+      <limit effort="100" lower="0.0" upper="0.044" velocity="0.2" />
       <mimic joint="${ee_prefix}finger_joint1" />
     </joint>

File: openarm_description/urdf/ee/openarm_hand_arguments.xacro (robot description, xacro)
@@ -12,5 +12,5 @@
   <xacro:arg name="rpy_ee" default= "0 0 0" />
   <!-- Position offset between ee frame and tcp frame -->
-  <xacro:arg name="tcp_xyz" default="0 0 0.1034" />
+  <xacro:arg name="tcp_xyz" default="0 0 0.0" />
   <!-- Rotation offset between ee frame and tcp frame -->
   <xacro:arg name="tcp_rpy" default="0 0 0" />

File: openarm_description/urdf/ee/openarm_hand_macro.xacro (robot description, xacro)
@@ -1,10 +1,4 @@
 <?xml version="1.0"?>
 <robot xmlns:xacro="http://www.ros.org/wiki/xacro">
-  <!-- ============================================================== -->
-  <!-- Macro to add an <inertial> tag based on yaml-load properties   -->
-  <!--                                                                -->
-  <!-- name:     Name of the end_effector (without prefix)              -->
-  <!-- ee_inertials: Dictionary of inertia properties (see inertial.yaml) -->
-  <!-- ============================================================== -->
   <xacro:macro name="ee-inertials" params="name ee_inertials:=^">
       <xacro:unless value="${name in ee_inertials}">${xacro.warning('No inertia properties defined for: ' + name)}</xacro:unless>
@@ -22,18 +16,9 @@
       </xacro:if>
   </xacro:macro>
-  <!-- ========================================================== -->
-  <!-- Macro to add a single link, both with                      -->
-  <!--  * detailed meshes for environmental collision checking    -->
-  <!--  * and coarse geometry models for self-collision checking  -->
-  <!--    (only if 'gazebo' param is set)                         -->
-  <!--                                                            -->
-  <!-- name:  Name of the end-effector (without prefix)             -->
-  <!-- rpy:   Rotation of the *_sc link relative to parent [rad]  -->
-  <!-- self_collision_geometries:  self <collision> models        -->
-  <!-- ========================================================== -->
-  <xacro:macro name="ee_link_with_sc" params="name prefix=${ee_prefix} rpy:='0 0 0' gazebo:=false">
+  <xacro:macro name="ee_link_with_sc" params="name prefix rpy:='0 0 0' gazebo:=false ee_kinematics_link">
     <!-- sub-link defining detailed meshes for collision with environment -->
     <link name="${prefix}${name}">
       <visual name="${prefix}${name}_visual">
+        <xacro:openarm-ee-kinematics-link config="${ee_kinematics_link}" name="${name}" />
         <geometry>
           <mesh filename="package://${description_pkg}/meshes/ee/${ee_type}/visual/${name}.dae" scale="0.001 0.001 0.001" />

File: openarm_description/urdf/robot/openarm_robot.xacro (robot description, xacro)
@@ -38,4 +38,7 @@
     <xacro:include filename="$(find openarm_description)/urdf/body/openarm_body_macro.xacro" />
     <xacro:include filename="$(find openarm_description)/urdf/body/openarm_body.xacro" />
+    <xacro:include filename="$(find openarm_description)/urdf/ee/openarm_hand.xacro" />
+    <xacro:include filename="$(find openarm_description)/urdf/ee/openarm_hand_macro.xacro" />
+    <xacro:include filename="$(find openarm_description)/urdf/ee/${ee_type}_arguments.xacro" />
     <xacro:property name="arm_prefix_modified" value="${'' if arm_prefix == '' else arm_prefix + '_'}" />
     <xacro:property name="body_prefix_modified" value="${'' if body_prefix == '' else body_prefix + '_'}" />
@@ -81,4 +84,34 @@
         kinematics="${kinematics}"
         kinematics_link="${kinematics_link}" />
+        <xacro:if value="${hand and ee_type == 'openarm_hand'}">
+            <xacro:openarm_hand
+                connected_to="left_${arm_type}_link8"
+                arm_type="${arm_type}"
+                arm_prefix="left_"
+                ee_type="${ee_type}"
+                ee_kinematics_link="${xacro.load_yaml('$(find openarm_description)/config/hand/openarm_hand/kinematics_link.yaml')}"
+                ee_inertials="${xacro.load_yaml('$(find openarm_description)/config/hand/openarm_hand/inertials.yaml')}"
+                rpy_ee="$(arg rpy_ee)"
+                xyz_ee="$(arg xyz_ee)"
+                tcp_xyz="$(arg tcp_xyz)"
+                tcp_rpy="$(arg tcp_rpy)"
+                gazebo="${gazebo}"
+                description_pkg="$(arg description_pkg)"
+            />
+            <xacro:openarm_hand
+                connected_to="right_${arm_type}_link8"
+                arm_type="${arm_type}"
+                arm_prefix="right_"
+                ee_type="${ee_type}"
+                ee_kinematics_link="${xacro.load_yaml('$(find openarm_description)/config/hand/openarm_hand/kinematics_link.yaml')}"
+                ee_inertials="${xacro.load_yaml('$(find openarm_description)/config/hand/openarm_hand/inertials.yaml')}"
+                rpy_ee="$(arg rpy_ee)"
+                xyz_ee="$(arg xyz_ee)"
+                tcp_xyz="$(arg tcp_xyz)"
+                tcp_rpy="$(arg tcp_rpy)"
+                gazebo="${gazebo}"
+                description_pkg="$(arg description_pkg)"
+            />
+          </xacro:if>
     </xacro:if>
     <xacro:if value="${not bimanual}">
@@ -97,7 +130,4 @@
         />
         <xacro:if value="${hand and ee_type == 'openarm_hand'}">
-        <xacro:include filename="$(find openarm_description)/urdf/ee/openarm_hand.xacro"/>
-        <xacro:include filename="$(find openarm_description)/urdf/ee/openarm_hand_macro.xacro" />
-        <xacro:include filename="$(find openarm_description)/urdf/ee/${ee_type}_arguments.xacro" />
         <xacro:property name="special_connection" value="$(arg special_connection)" />
         <xacro:property name="connection" value="${special_connection if special_connection != '' else arm_type + '_link8'}" />
@@ -108,5 +138,5 @@
             ee_type="${ee_type}"
             ee_kinematics_link="${xacro.load_yaml('$(find openarm_description)/config/hand/openarm_hand/kinematics_link.yaml')}"
-            ee_inertials="${xacro.load_yaml('$(find openarm_description)/config/hand/$(arg ee_type)/hand_inertials.yaml')}"
+            ee_inertials="${xacro.load_yaml('$(find openarm_description)/config/hand/openarm_hand/inertials.yaml')}"
             rpy_ee="$(arg rpy_ee)"
             xyz_ee="$(arg xyz_ee)"
@@ -117,8 +147,5 @@
         />
         </xacro:if>
-        <xacro:if value="${hand and ee_type != 'none' and ee_type != 'openarm_hand'}">
-        <xacro:include filename="$(find openarm_description)/urdf/ee/ee_with_one_link.xacro"/>
-        <xacro:include filename="$(find openarm_description)/urdf/ee/openarm_hand_macro.xacro" />
-        <xacro:include filename="$(find openarm_description)/urdf/ee/${ee_type}_arguments.xacro" />
+        <!-- <xacro:if value="${hand and ee_type != 'none' and ee_type != 'openarm_hand'}">
         <xacro:property name="special_connection" value="$(arg special_connection)" />
         <xacro:property name="connection" value="${special_connection if special_connection == '' else arm_type + '_link8'}" />
@@ -137,5 +164,5 @@
             description_pkg="$(arg description_pkg)"
         />
-        </xacro:if>
+        </xacro:if> -->
         </xacro:if>
         <!-- <xacro:if value="${gazebo}">

File: openarm_description/urdf/robot/v10.urdf.xacro (robot description, xacro)
@@ -9,10 +9,9 @@
   <xacro:arg name="arm_type" default="v10" />
   <xacro:arg name="body_type" default="v10" />
+  <xacro:arg name="ee_type" default="openarm_hand" />
   <!-- Don't print a prefix for joints, visuals, and links? -->
   <xacro:arg name="no_prefix" default="false"/>
   <!-- Should an end-effector be mounted at the flange?" -->
   <xacro:arg name="hand" default="true" />
-  <!-- Which end-effector would be mounted at the flange?" -->
-  <xacro:arg name="ee_type" default="openarm_hand" />
   <!-- Is the robot being simulated in gazebo?" -->
   <xacro:arg name="gazebo" default="false" />
