Commit message: add: body stl

File: openarm_description/urdf/body/openarm_body_macro.xacro (robot description, xacro)
@@ -38,5 +38,5 @@
         <xacro:openarm-body-kinematics config="${kinematics_link}" name="${name}" />
         <geometry>
-          <mesh filename="package://${description_pkg}/meshes/body/${body_type}/visual/${name}.stl" scale="0.001 0.001 0.001" />
+          <mesh filename="package://${description_pkg}/meshes/body/${body_type}/visual/${name}.dae" scale="0.001 0.001 0.001" />
         </geometry>
       </visual>

File: openarm_description/urdf/robot/v10.urdf.xacro (robot description, xacro)
@@ -35,7 +35,7 @@
   <xacro:arg name="bimanual" default="false" />
   <!-- used in bimanual -->
-  <xacro:arg name="right_arm_base_xyz" default="0.0 -0.07 0.83" />
+  <xacro:arg name="right_arm_base_xyz" default="0.0 -0.031 0.698" />
   <xacro:arg name="right_arm_base_rpy" default="1.5708 0 0" />
-  <xacro:arg name="left_arm_base_xyz" default="0.0 0.07 0.83" />
+  <xacro:arg name="left_arm_base_xyz" default="0.0 0.031 0.698" />
   <xacro:arg name="left_arm_base_rpy" default="-1.5708 0 0" />
   <xacro:openarm_robot
