Commit message: add: body

File: openarm_description/urdf/arm/openarm_arm.xacro (robot description, xacro)
@@ -1,5 +1,5 @@
 <?xml version='1.0' encoding='utf-8'?>
 <robot xmlns:xacro="http://www.ros.org/wiki/xacro" name="openarm">
-  <xacro:include filename="$(find openarm_description)/urdf/common/openarm_macro.xacro" />
+  <xacro:include filename="$(find openarm_description)/urdf/arm/openarm_macro.xacro" />
   <!-- arm_type: Namespace of the robot arm. Serves to differentiate between arms in case of multiple instances. -->
   <!-- joint_limits: description of the joint limits that comes from a YAML file. Example definition: ${xacro.load_yaml('$(find openarm_description)/robots/fr3/joint_limits.yaml')} -->

File: openarm_description/urdf/robot/openarm_robot.xacro (robot description, xacro)
@@ -1,35 +1,52 @@
 <?xml version='1.0' encoding='utf-8'?>
 <robot xmlns:xacro="http://www.ros.org/wiki/xacro">
-  <xacro:macro name="openarm_robot"
-              params="arm_type
-                      joint_limits
-                      kinematics
-                      kinematics_link
-                      inertials
-                      parent:='world'
-                      xyz:='0 0 0'
-                      rpy:='0 0 0'
-                      hand:='true'
-                      ee_type:=none
-                      gazebo:='false'
-                      ros2_control:=false
-                      can:=''
-                      use_fake_hardware:=false
-                      fake_sensor_commands:=false
-                      gazebo_effort:=false
-                      no_prefix:='false'
-                      arm_prefix:=''
-                      connected_to:='base'
-                      bimanual:=false">
-    <xacro:include filename="$(find openarm_description)/urdf/common/openarm_macro.xacro" />
-    <xacro:include filename="$(find openarm_description)/urdf/common/openarm_arm.xacro" />
-    <xacro:include filename="$(find openarm_description)/urdf_body/common/openarm_body.xacro" />
+    <xacro:macro name="openarm_robot"
+    params="arm_type
+            joint_limits
+            kinematics
+            kinematics_link
+            inertials
+            body_type
+            body_inertials
+            body_kinematics
+            body_kinematics_link
+            parent:='world'
+            xyz:='0 0 0'
+            rpy:='0 0 0'
+            hand:='true'
+            ee_type:=none
+            gazebo:='false'
+            ros2_control:=false
+            can:=''
+            use_fake_hardware:=false
+            fake_sensor_commands:=false
+            gazebo_effort:=false
+            no_prefix:='false'
+            arm_prefix:=''
+            body_prefix:=''
+            arm_connected_to='base'
+            body_connected_to='world'
+            bimanual:=true">
+    <xacro:include filename="$(find openarm_description)/urdf/arm/openarm_macro.xacro" />
+    <xacro:include filename="$(find openarm_description)/urdf/arm/openarm_arm.xacro" />
+    <xacro:include filename="$(find openarm_description)/urdf/body/openarm_body_macro.xacro" />
+    <xacro:include filename="$(find openarm_description)/urdf/body/openarm_body.xacro" />
     <xacro:property name="arm_prefix_modified" value="${'' if arm_prefix == '' else arm_prefix + '_'}" />
-    <xacro:openarm_body
-    body_type="v10"
-    body_inertials="${xacro.load_yaml('$(find openarm_description)/config/body/v10/inertials.yaml')}"
-    gazebo="false"
-    description_pkg="openarm_description"
-  />
+    <xacro:property name="body_prefix_modified" value="${'' if body_prefix == '' else body_prefix + '_'}" />
+    <xacro:if value="${bimanual}">
+        <xacro:openarm_body
+        body_type="${body_type}"
+        body_prefix="${body_prefix_modified}"
+        no_prefix="${no_prefix}"
+        description_pkg="openarm_description"
+        connected_to="${body_connected_to}"
+        xyz="${xyz}"
+        rpy="${rpy}"
+        gazebo="${gazebo}"
+        inertials="${body_inertials}"
+        kinematics="${body_kinematics}"
+        kinematics_link="${body_kinematics_link}" />
+    </xacro:if>
+ <xacro:if value="${not bimanual}">
     <xacro:openarm_arm
       arm_type="${arm_type}"
@@ -43,16 +60,10 @@
       kinematics_link="${kinematics_link}"
       inertials="${inertials}"
-      connected_to="${connected_to}"
+      connected_to="${arm_connected_to}"
     />
     <xacro:if value="${hand and ee_type == 'openarm_hand'}">
-      <xacro:include filename="$(find openarm_description)/urdf_end_effector/common/openarm_hand.xacro"/>
-      <xacro:include filename="$(find openarm_description)/urdf_end_effector/common/openarm_hand_macro.xacro" />
-      <xacro:include filename="$(find openarm_description)/urdf_end_effector/${ee_type}/${ee_type}_arguments.xacro" />
-      <!-- <xacro:if value="${arm_type == 'v10'}">
-        <xacro:property name="ee_color" value="black" />
-      </xacro:if>
-      <xacro:if value="${arm_type == 'v10' or arm_type == 'v10'}">
-        <xacro:property name="ee_color" value="white" />
-      </xacro:if> -->
+      <xacro:include filename="$(find openarm_description)/urdf/ee/openarm_hand.xacro"/>
+      <xacro:include filename="$(find openarm_description)/urdf/ee/openarm_hand_macro.xacro" />
+      <xacro:include filename="$(find openarm_description)/urdf/${ee_type}_arguments.xacro" />
       <xacro:property name="special_connection" value="$(arg special_connection)" />
       <xacro:property name="connection" value="${special_connection if special_connection != '' else arm_type + '_link8'}" />
@@ -72,7 +83,7 @@
     </xacro:if>
     <xacro:if value="${hand and ee_type != 'none' and ee_type != 'openarm_hand'}">
-      <xacro:include filename="$(find openarm_description)/urdf_end_effector/common/ee_with_one_link.xacro"/>
-      <xacro:include filename="$(find openarm_description)/urdf_end_effector/common/openarm_hand_macro.xacro" />
-      <xacro:include filename="$(find openarm_description)/urdf_end_effector/$(arg ee_type)/${ee_type}_arguments.xacro" />
+      <xacro:include filename="$(find openarm_description)/urdf/ee/ee_with_one_link.xacro"/>
+      <xacro:include filename="$(find openarm_description)/urdf/ee/openarm_hand_macro.xacro" />
+      <xacro:include filename="$(find openarm_description)/urdf/${ee_type}_arguments.xacro" />
       <xacro:property name="special_connection" value="$(arg special_connection)" />
       <xacro:property name="connection" value="${special_connection if special_connection == '' else arm_type + '_link8'}" />
@@ -91,8 +102,7 @@
       />
     </xacro:if>
-    <!-- Definition of additional Gazebo tags -->
-    <xacro:if value="${gazebo}">
+    </xacro:if>
+    <!-- <xacro:if value="${gazebo}">
       <xacro:if value="${parent != ''}">
-        <!-- Gazebo requires a joint to a link called "world" for statically mounted robots -->
         <xacro:if value="${parent == 'world'}">
           <link name="${parent}" />
@@ -133,5 +143,4 @@
         <xacro:gazebo-joint joint="${arm_type}_finger_joint1" transmission="hardware_interface/EffortJointInterface" />
         <xacro:gazebo-joint joint="${arm_type}_finger_joint2" transmission="hardware_interface/EffortJointInterface" />
-        <!-- Friction specific material for Rubber/Rubber contact -->
         <xacro:gazebo-friction link="${arm_type}_leftfinger" mu="1.13" />
         <xacro:gazebo-friction link="${arm_type}_rightfinger" mu="1.13" />
@@ -139,5 +148,5 @@
     </xacro:if>
     <xacro:if value="${ros2_control}">
-      <xacro:include filename="$(find openarm_description)/urdf/common/openarm_arm.ros2_control.xacro"/>
+      <xacro:include filename="$(find openarm_description)/urdf/ros2_control/openarm_arm.ros2_control.xacro"/>
       <xacro:openarm_arm_ros2_control
           arm_type="${arm_type}"
@@ -151,5 +160,5 @@
           multi_arm="$(arg multi_arm)"
       />
-    </xacro:if>
+    </xacro:if> -->
   </xacro:macro>
 </robot>

File: openarm_description/urdf/robot/v10.urdf.xacro (robot description, xacro)
@@ -1,5 +1,5 @@
 <?xml version='1.0' encoding='utf-8'?>
 <robot xmlns:xacro="http://www.ros.org/wiki/xacro" name="openarm">
-  <xacro:include filename="$(find openarm_description)/urdf/common/openarm_robot.xacro"/>
+  <xacro:include filename="$(find openarm_description)/urdf/robot/openarm_robot.xacro"/>
   <!--
     DEPRECATION NOTICE
@@ -8,9 +8,9 @@
   -->
   <xacro:arg name="arm_type" default="v10" />
-  <!-- <xacro:arg name="body_type" default="v10" /> -->
+  <xacro:arg name="body_type" default="v10" />
   <!-- Don't print a prefix for joints, visuals, and links? -->
   <xacro:arg name="no_prefix" default="false"/>
   <!-- Should an end-effector be mounted at the flange?" -->
-  <xacro:arg name="hand" default="true" />
+  <xacro:arg name="hand" default="false" />
   <!-- Which end-effector would be mounted at the flange?" -->
   <xacro:arg name="ee_type" default="openarm_hand" />
@@ -35,21 +35,27 @@
   <!-- For a multi arm setup, we need a threaded robot running async-->
   <xacro:arg name="bimanual" default="false" />
-  <xacro:openarm_robot arm_type="v10"
-                      joint_limits="${xacro.load_yaml('$(find openarm_description)/config/v10/joint_limits.yaml')}"
-                      inertials="${xacro.load_yaml('$(find openarm_description)/config/v10/inertials.yaml')}"
-                      kinematics="${xacro.load_yaml('$(find openarm_description)/config/v10/kinematics.yaml')}"
-                      kinematics_link="${xacro.load_yaml('$(find openarm_description)/config/v10/kinematics_link.yaml')}"
-                      gazebo="$(arg gazebo)"
-                      hand="$(arg hand)"
-                      ee_type="$(arg ee_type)"
-                      ros2_control="$(arg ros2_control)"
-                      can="$(arg can)"
-                      use_fake_hardware="$(arg use_fake_hardware)"
-                      fake_sensor_commands="$(arg fake_sensor_commands)"
-                      gazebo_effort="$(arg gazebo_effort)"
-                      no_prefix="$(arg no_prefix)"
-                      arm_prefix= ""
-                      connected_to= "base"
-                      bimanual= "$(arg bimanual)">
-  </xacro:openarm_robot>
+  <xacro:openarm_robot
+  arm_type="v10"
+  body_type="v10"
+  joint_limits="${xacro.load_yaml('$(find openarm_description)/config/v10/joint_limits.yaml')}"
+  inertials="${xacro.load_yaml('$(find openarm_description)/config/v10/inertials.yaml')}"
+  kinematics="${xacro.load_yaml('$(find openarm_description)/config/v10/kinematics.yaml')}"
+  kinematics_link="${xacro.load_yaml('$(find openarm_description)/config/v10/kinematics_link.yaml')}"
+  body_inertials="${xacro.load_yaml('$(find openarm_description)/config/body/v10/inertials.yaml')}"
+  body_kinematics="${xacro.load_yaml('$(find openarm_description)/config/body/v10/kinematics.yaml')}"
+  body_kinematics_link="${xacro.load_yaml('$(find openarm_description)/config/body/v10/kinematics.yaml')}"
+  gazebo="$(arg gazebo)"
+  hand="$(arg hand)"
+  ee_type="$(arg ee_type)"
+  ros2_control="$(arg ros2_control)"
+  can="$(arg can)"
+  use_fake_hardware="$(arg use_fake_hardware)"
+  fake_sensor_commands="$(arg fake_sensor_commands)"
+  gazebo_effort="$(arg gazebo_effort)"
+  no_prefix="$(arg no_prefix)"
+  arm_prefix=""
+  body_prefix=""
+  arm_connected_to="base"
+  body_connected_to="world"
+  bimanual="$(arg bimanual)" />
 </robot>
