Commit message: add: bimanual

File: openarm_description/urdf/arm/openarm_arm.xacro (robot description, xacro)
@@ -12,7 +12,7 @@
       <xacro:property name="connected_to" value="" />
     </xacro:if>
-    <xacro:unless value="${not connected_to}">
-      <link name="${connected_to}">
-      </link>
+    <xacro:unless value="${connected_to == ''}">
+      <!-- <link name="${connected_to}">
+      </link> -->
       <joint name="${prefix}${connected_to}_joint" type="fixed">
         <parent link="${connected_to}"/>

File: openarm_description/urdf/body/openarm_body.xacro (robot description, xacro)
@@ -30,13 +30,13 @@
     </xacro:macro>
     <!-- for bimanual right side-->
-    <!-- <joint name="${body_type}_to_right_${arm_type}_joint" type="fixed">
+    <!-- <joint name="${body_type}_body_to_right_${arm_type}_joint" type="fixed">
       <origin xyz="0.3 -0.2 0.4" rpy="0 0 0" />
-      <parent link="${body_type}_body_link0" />
+      <parent link="body_link0" />
       <child link="right_${arm_type}_link0" />
     </joint> -->
     <!-- for bimanual left side-->
-    <!-- <joint name="${body_type}_to_left_${arm_type}_joint" type="fixed">
+    <!-- <joint name="${body_type}_body_to_left_${arm_type}_joint" type="fixed">
       <origin xyz="0.3 0.2 0.4" rpy="0 0 0" />
-      <parent link="${body_type}_body_link0" />
+      <parent link="body_link0" />
       <child link="left_${arm_type}_link0" />
     </joint> -->

File: openarm_description/urdf/robot/openarm_robot.xacro (robot description, xacro)
@@ -27,5 +27,10 @@
             arm_connected_to='base'
             body_connected_to='world'
-            bimanual:=true">
+            bimanual:=true
+            right_arm_base_xyz='0 0 0'
+            left_arm_base_xyz='0 0 0'
+            right_arm_base_rpy='0 0 0'
+            left_arm_base_rpy='0 0 0' "
+            >
     <xacro:include filename="$(find openarm_description)/urdf/arm/openarm_macro.xacro" />
     <xacro:include filename="$(find openarm_description)/urdf/arm/openarm_arm.xacro" />
@@ -47,118 +52,146 @@
         kinematics="${body_kinematics}"
         kinematics_link="${body_kinematics_link}" />
+        <!-- left arm -->
+        <xacro:openarm_arm
+        arm_type="${arm_type}"
+        arm_prefix="left_"
+        no_prefix="false"
+        description_pkg="openarm_description"
+        connected_to="${body_type}_body_link0"
+        xyz="${left_arm_base_xyz}"
+        rpy="${left_arm_base_rpy}"
+        gazebo="${gazebo}"
+        joint_limits="${joint_limits}"
+        inertials="${inertials}"
+        kinematics="${kinematics}"
+        kinematics_link="${kinematics_link}" />
+        <!-- right arm -->
+        <xacro:openarm_arm
+        arm_type="${arm_type}"
+        arm_prefix="right_"
+        no_prefix="false"
+        description_pkg="openarm_description"
+        connected_to="${body_type}_body_link0"
+        xyz="${right_arm_base_xyz}"
+        rpy="${right_arm_base_rpy}"
+        gazebo="${gazebo}"
+        joint_limits="${joint_limits}"
+        inertials="${inertials}"
+        kinematics="${kinematics}"
+        kinematics_link="${kinematics_link}" />
     </xacro:if>
- <xacro:if value="${not bimanual}">
-    <xacro:openarm_arm
-      arm_type="${arm_type}"
-      arm_prefix="${arm_prefix_modified}"
-      no_prefix="${no_prefix}"
-      xyz="${xyz}"
-      rpy="${rpy}"
-      gazebo="${gazebo}"
-      joint_limits="${joint_limits}"
-      kinematics="${kinematics}"
-      kinematics_link="${kinematics_link}"
-      inertials="${inertials}"
-      connected_to="${arm_connected_to}"
-    />
-    <xacro:if value="${hand and ee_type == 'openarm_hand'}">
-      <xacro:include filename="$(find openarm_description)/urdf/ee/openarm_hand.xacro"/>
-      <xacro:include filename="$(find openarm_description)/urdf/ee/openarm_hand_macro.xacro" />
-      <xacro:include filename="$(find openarm_description)/urdf/${ee_type}_arguments.xacro" />
-      <xacro:property name="special_connection" value="$(arg special_connection)" />
-      <xacro:property name="connection" value="${special_connection if special_connection != '' else arm_type + '_link8'}" />
-      <xacro:openarm_hand
-        connected_to="${arm_prefix_modified}${connection}"
+    <xacro:if value="${not bimanual}">
+        <xacro:openarm_arm
         arm_type="${arm_type}"
         arm_prefix="${arm_prefix_modified}"
-        ee_type="${ee_type}"
-        ee_inertials="${xacro.load_yaml('$(find openarm_description)/config/hand/$(arg ee_type)/hand_inertials.yaml')}"
-        rpy_ee="$(arg rpy_ee)"
-        xyz_ee="$(arg xyz_ee)"
-        tcp_xyz="$(arg tcp_xyz)"
-        tcp_rpy="$(arg tcp_rpy)"
+        no_prefix="${no_prefix}"
+        xyz="${xyz}"
+        rpy="${rpy}"
         gazebo="${gazebo}"
-        description_pkg="$(arg description_pkg)"
-      />
-    </xacro:if>
-    <xacro:if value="${hand and ee_type != 'none' and ee_type != 'openarm_hand'}">
-      <xacro:include filename="$(find openarm_description)/urdf/ee/ee_with_one_link.xacro"/>
-      <xacro:include filename="$(find openarm_description)/urdf/ee/openarm_hand_macro.xacro" />
-      <xacro:include filename="$(find openarm_description)/urdf/${ee_type}_arguments.xacro" />
-      <xacro:property name="special_connection" value="$(arg special_connection)" />
-      <xacro:property name="connection" value="${special_connection if special_connection == '' else arm_type + '_link8'}" />
-      <xacro:ee_with_one_link
-        connected_to="${arm_prefix_modified}${connection}"
-        arm_type="${arm_type}"
-        arm_prefix="${arm_prefix_modified}"
-        ee_type="${ee_type}"
-        ee_inertials="${xacro.load_yaml('$(find openarm_description)/config/hand/$(arg ee_type)_inertials.yaml')}"
-        rpy_ee="$(arg rpy_ee)"
-        xyz_ee="$(arg xyz_ee)"
-        tcp_xyz="$(arg tcp_xyz)"
-        tcp_rpy="$(arg tcp_rpy)"
-        gazebo="${gazebo}"
-        description_pkg="$(arg description_pkg)"
-      />
-    </xacro:if>
-    </xacro:if>
-    <!-- <xacro:if value="${gazebo}">
-      <xacro:if value="${parent != ''}">
-        <xacro:if value="${parent == 'world'}">
-          <link name="${parent}" />
+        joint_limits="${joint_limits}"
+        kinematics="${kinematics}"
+        kinematics_link="${kinematics_link}"
+        inertials="${inertials}"
+        connected_to=""
+        />
+        <xacro:if value="${hand and ee_type == 'openarm_hand'}">
+        <xacro:include filename="$(find openarm_description)/urdf/ee/openarm_hand.xacro"/>
+        <xacro:include filename="$(find openarm_description)/urdf/ee/openarm_hand_macro.xacro" />
+        <xacro:include filename="$(find openarm_description)/urdf/${ee_type}_arguments.xacro" />
+        <xacro:property name="special_connection" value="$(arg special_connection)" />
+        <xacro:property name="connection" value="${special_connection if special_connection != '' else arm_type + '_link8'}" />
+        <xacro:openarm_hand
+            connected_to="${arm_prefix_modified}${connection}"
+            arm_type="${arm_type}"
+            arm_prefix="${arm_prefix_modified}"
+            ee_type="${ee_type}"
+            ee_inertials="${xacro.load_yaml('$(find openarm_description)/config/hand/$(arg ee_type)/hand_inertials.yaml')}"
+            rpy_ee="$(arg rpy_ee)"
+            xyz_ee="$(arg xyz_ee)"
+            tcp_xyz="$(arg tcp_xyz)"
+            tcp_rpy="$(arg tcp_rpy)"
+            gazebo="${gazebo}"
+            description_pkg="$(arg description_pkg)"
+        />
         </xacro:if>
-        <joint name="${parent}_joint" type="fixed">
-          <origin xyz="${xyz}" rpy="${rpy}" />
-          <parent link="${parent}" />
-          <child  link="${arm_type}_link0" />
-        </joint>
-    </xacro:if>
-      <xacro:gazebo-joint joint="${arm_type}_joint1" transmission="hardware_interface/PositionJointInterface" />
-      <xacro:gazebo-joint joint="${arm_type}_joint2" transmission="hardware_interface/PositionJointInterface" />
-      <xacro:gazebo-joint joint="${arm_type}_joint3" transmission="hardware_interface/PositionJointInterface" />
-      <xacro:gazebo-joint joint="${arm_type}_joint4" transmission="hardware_interface/PositionJointInterface" />
-      <xacro:gazebo-joint joint="${arm_type}_joint5" transmission="hardware_interface/PositionJointInterface" />
-      <xacro:gazebo-joint joint="${arm_type}_joint6" transmission="hardware_interface/PositionJointInterface" />
-      <xacro:gazebo-joint joint="${arm_type}_joint7" transmission="hardware_interface/PositionJointInterface" />
-      <xacro:gazebo-joint joint="${arm_type}_joint1" transmission="hardware_interface/VelocityJointInterface" />
-      <xacro:gazebo-joint joint="${arm_type}_joint2" transmission="hardware_interface/VelocityJointInterface" />
-      <xacro:gazebo-joint joint="${arm_type}_joint3" transmission="hardware_interface/VelocityJointInterface" />
-      <xacro:gazebo-joint joint="${arm_type}_joint4" transmission="hardware_interface/VelocityJointInterface" />
-      <xacro:gazebo-joint joint="${arm_type}_joint5" transmission="hardware_interface/VelocityJointInterface" />
-      <xacro:gazebo-joint joint="${arm_type}_joint6" transmission="hardware_interface/VelocityJointInterface" />
-      <xacro:gazebo-joint joint="${arm_type}_joint7" transmission="hardware_interface/VelocityJointInterface" />
-      <xacro:gazebo-joint joint="${arm_type}_joint1" transmission="hardware_interface/EffortJointInterface" />
-      <xacro:gazebo-joint joint="${arm_type}_joint2" transmission="hardware_interface/EffortJointInterface" />
-      <xacro:gazebo-joint joint="${arm_type}_joint3" transmission="hardware_interface/EffortJointInterface" />
-      <xacro:gazebo-joint joint="${arm_type}_joint4" transmission="hardware_interface/EffortJointInterface" />
-      <xacro:gazebo-joint joint="${arm_type}_joint5" transmission="hardware_interface/EffortJointInterface" />
-      <xacro:gazebo-joint joint="${arm_type}_joint6" transmission="hardware_interface/EffortJointInterface" />
-      <xacro:gazebo-joint joint="${arm_type}_joint7" transmission="hardware_interface/EffortJointInterface" />
-      <xacro:transmission-openarm-state arm_type="${arm_type}" />
-      <xacro:transmission-openarm-model arm_type="${arm_type}"
-         root="${arm_type}_joint1"
-         tip="${arm_type}_joint8"
-       />
-      <xacro:if value="${ee_type == 'openarm_hand'}">
-        <xacro:gazebo-joint joint="${arm_type}_finger_joint1" transmission="hardware_interface/EffortJointInterface" />
-        <xacro:gazebo-joint joint="${arm_type}_finger_joint2" transmission="hardware_interface/EffortJointInterface" />
-        <xacro:gazebo-friction link="${arm_type}_leftfinger" mu="1.13" />
-        <xacro:gazebo-friction link="${arm_type}_rightfinger" mu="1.13" />
-      </xacro:if>
-    </xacro:if>
-    <xacro:if value="${ros2_control}">
-      <xacro:include filename="$(find openarm_description)/urdf/ros2_control/openarm_arm.ros2_control.xacro"/>
-      <xacro:openarm_arm_ros2_control
-          arm_type="${arm_type}"
-          can="${can}"
-          use_fake_hardware="$(arg use_fake_hardware)"
-          fake_sensor_commands="$(arg fake_sensor_commands)"
-          gazebo="$(arg gazebo)"
-          hand="$(arg hand)"
-          gazebo_effort="$(arg gazebo_effort)"
-          arm_prefix="${arm_prefix}"
-          multi_arm="$(arg multi_arm)"
-      />
-    </xacro:if> -->
+        <xacro:if value="${hand and ee_type != 'none' and ee_type != 'openarm_hand'}">
+        <xacro:include filename="$(find openarm_description)/urdf/ee/ee_with_one_link.xacro"/>
+        <xacro:include filename="$(find openarm_description)/urdf/ee/openarm_hand_macro.xacro" />
+        <xacro:include filename="$(find openarm_description)/urdf/${ee_type}_arguments.xacro" />
+        <xacro:property name="special_connection" value="$(arg special_connection)" />
+        <xacro:property name="connection" value="${special_connection if special_connection == '' else arm_type + '_link8'}" />
+        <xacro:ee_with_one_link
+            connected_to="${arm_prefix_modified}${connection}"
+            arm_type="${arm_type}"
+            arm_prefix="${arm_prefix_modified}"
+            ee_type="${ee_type}"
+            ee_inertials="${xacro.load_yaml('$(find openarm_description)/config/hand/$(arg ee_type)_inertials.yaml')}"
+            rpy_ee="$(arg rpy_ee)"
+            xyz_ee="$(arg xyz_ee)"
+            tcp_xyz="$(arg tcp_xyz)"
+            tcp_rpy="$(arg tcp_rpy)"
+            gazebo="${gazebo}"
+            description_pkg="$(arg description_pkg)"
+        />
+        </xacro:if>
+        </xacro:if>
+        <!-- <xacro:if value="${gazebo}">
+        <xacro:if value="${parent != ''}">
+            <xacro:if value="${parent == 'world'}">
+            <link name="${parent}" />
+            </xacro:if>
+            <joint name="${parent}_joint" type="fixed">
+            <origin xyz="${xyz}" rpy="${rpy}" />
+            <parent link="${parent}" />
+            <child  link="${arm_type}_link0" />
+            </joint>
+        </xacro:if>
+        <xacro:gazebo-joint joint="${arm_type}_joint1" transmission="hardware_interface/PositionJointInterface" />
+        <xacro:gazebo-joint joint="${arm_type}_joint2" transmission="hardware_interface/PositionJointInterface" />
+        <xacro:gazebo-joint joint="${arm_type}_joint3" transmission="hardware_interface/PositionJointInterface" />
+        <xacro:gazebo-joint joint="${arm_type}_joint4" transmission="hardware_interface/PositionJointInterface" />
+        <xacro:gazebo-joint joint="${arm_type}_joint5" transmission="hardware_interface/PositionJointInterface" />
+        <xacro:gazebo-joint joint="${arm_type}_joint6" transmission="hardware_interface/PositionJointInterface" />
+        <xacro:gazebo-joint joint="${arm_type}_joint7" transmission="hardware_interface/PositionJointInterface" />
+        <xacro:gazebo-joint joint="${arm_type}_joint1" transmission="hardware_interface/VelocityJointInterface" />
+        <xacro:gazebo-joint joint="${arm_type}_joint2" transmission="hardware_interface/VelocityJointInterface" />
+        <xacro:gazebo-joint joint="${arm_type}_joint3" transmission="hardware_interface/VelocityJointInterface" />
+        <xacro:gazebo-joint joint="${arm_type}_joint4" transmission="hardware_interface/VelocityJointInterface" />
+        <xacro:gazebo-joint joint="${arm_type}_joint5" transmission="hardware_interface/VelocityJointInterface" />
+        <xacro:gazebo-joint joint="${arm_type}_joint6" transmission="hardware_interface/VelocityJointInterface" />
+        <xacro:gazebo-joint joint="${arm_type}_joint7" transmission="hardware_interface/VelocityJointInterface" />
+        <xacro:gazebo-joint joint="${arm_type}_joint1" transmission="hardware_interface/EffortJointInterface" />
+        <xacro:gazebo-joint joint="${arm_type}_joint2" transmission="hardware_interface/EffortJointInterface" />
+        <xacro:gazebo-joint joint="${arm_type}_joint3" transmission="hardware_interface/EffortJointInterface" />
+        <xacro:gazebo-joint joint="${arm_type}_joint4" transmission="hardware_interface/EffortJointInterface" />
+        <xacro:gazebo-joint joint="${arm_type}_joint5" transmission="hardware_interface/EffortJointInterface" />
+        <xacro:gazebo-joint joint="${arm_type}_joint6" transmission="hardware_interface/EffortJointInterface" />
+        <xacro:gazebo-joint joint="${arm_type}_joint7" transmission="hardware_interface/EffortJointInterface" />
+        <xacro:transmission-openarm-state arm_type="${arm_type}" />
+        <xacro:transmission-openarm-model arm_type="${arm_type}"
+            root="${arm_type}_joint1"
+            tip="${arm_type}_joint8"
+        />
+        <xacro:if value="${ee_type == 'openarm_hand'}">
+            <xacro:gazebo-joint joint="${arm_type}_finger_joint1" transmission="hardware_interface/EffortJointInterface" />
+            <xacro:gazebo-joint joint="${arm_type}_finger_joint2" transmission="hardware_interface/EffortJointInterface" />
+            <xacro:gazebo-friction link="${arm_type}_leftfinger" mu="1.13" />
+            <xacro:gazebo-friction link="${arm_type}_rightfinger" mu="1.13" />
+        </xacro:if>
+        </xacro:if>
+        <xacro:if value="${ros2_control}">
+        <xacro:include filename="$(find openarm_description)/urdf/ros2_control/openarm_arm.ros2_control.xacro"/>
+        <xacro:openarm_arm_ros2_control
+            arm_type="${arm_type}"
+            can="${can}"
+            use_fake_hardware="$(arg use_fake_hardware)"
+            fake_sensor_commands="$(arg fake_sensor_commands)"
+            gazebo="$(arg gazebo)"
+            hand="$(arg hand)"
+            gazebo_effort="$(arg gazebo_effort)"
+            arm_prefix="${arm_prefix}"
+            multi_arm="$(arg multi_arm)"
+        />
+        </xacro:if> -->
   </xacro:macro>
 </robot>

File: openarm_description/urdf/robot/v10.urdf.xacro (robot description, xacro)
@@ -34,5 +34,9 @@
   <xacro:arg name="gazebo_effort" default="false" />
   <!-- For a multi arm setup, we need a threaded robot running async-->
-  <xacro:arg name="bimanual" default="false" />
+  <xacro:arg name="bimanual" default="true" />
+  <xacro:arg name="right_arm_base_xyz" default="0.0 0.07 0.83" />
+  <xacro:arg name="right_arm_base_rpy" default="-1.5708 0 0" />
+  <xacro:arg name="left_arm_base_xyz" default="0.0 -0.07 0.83" />
+  <xacro:arg name="left_arm_base_rpy" default="1.5708 0 0" />
   <xacro:openarm_robot
   arm_type="v10"
@@ -58,4 +62,9 @@
   arm_connected_to="base"
   body_connected_to="world"
-  bimanual="$(arg bimanual)" />
+  bimanual="$(arg bimanual)"
+  right_arm_base_xyz="$(arg right_arm_base_xyz)"
+  left_arm_base_xyz="$(arg left_arm_base_rpy)"
+  right_arm_base_rpy="$(arg right_arm_base_rpy)"
+  left_arm_base_rpy="$(arg left_arm_base_rpy)"
+  />
 </robot>
