Commit message: fix: hand dae

File: openarm_description/urdf/arm/openarm_arm.xacro (robot description, xacro)
@@ -9,4 +9,10 @@
     <!-- Define a property that defaults to 'arm_prefix_arm_type' concatenated with an underscore if 'no_prefix' is not set -->
     <xacro:property name="prefix" value="${'' if no_prefix else arm_prefix + arm_type + '_'}" />
+    <xacro:if value="${arm_prefix == 'right_'}">
+      <xacro:property name="reflect" value="-1" />
+    </xacro:if>
+    <xacro:unless value="${arm_prefix == 'right_'}">
+      <xacro:property name="reflect" value="1" />
+    </xacro:unless>
     <xacro:if value="${gazebo}">
       <xacro:property name="connected_to" value="" />
@@ -21,6 +27,6 @@
       </joint>
     </xacro:unless>
-    <xacro:link_with_sc no_prefix="${no_prefix}" name="link0" gazebo="${gazebo}" kinematics_link="${kinematics_link}"/>
-    <xacro:link_with_sc no_prefix="${no_prefix}" name="link1" gazebo="${gazebo}" kinematics_link="${kinematics_link}"/>
+    <xacro:link_with_sc no_prefix="${no_prefix}" name="link0" gazebo="${gazebo}" kinematics_link="${kinematics_link}" reflect="${reflect}"/>
+    <xacro:link_with_sc no_prefix="${no_prefix}" name="link1" gazebo="${gazebo}" kinematics_link="${kinematics_link}" reflect="${reflect}"/>
     <joint name="${prefix}joint1" type="revolute">
       <xacro:openarm-kinematics name="joint1" config="${kinematics}" />
@@ -30,5 +36,5 @@
       <xacro:openarm-limits name="joint1" config="${joint_limits}" />
     </joint>
-    <xacro:link_with_sc no_prefix="${no_prefix}" name="link2" gazebo="${gazebo}" kinematics_link="${kinematics_link}"/>
+    <xacro:link_with_sc no_prefix="${no_prefix}" name="link2" gazebo="${gazebo}" kinematics_link="${kinematics_link}" reflect="${reflect}"/>
     <joint name="${prefix}joint2" type="revolute">
       <xacro:openarm-kinematics name="joint2" config="${kinematics}" />
@@ -38,5 +44,5 @@
       <xacro:openarm-limits name="joint2" config="${joint_limits}" />
     </joint>
-    <xacro:link_with_sc no_prefix="${no_prefix}" name="link3" gazebo="${gazebo}" kinematics_link="${kinematics_link}" />
+    <xacro:link_with_sc no_prefix="${no_prefix}" name="link3" gazebo="${gazebo}" kinematics_link="${kinematics_link}" reflect="${reflect}"/>
     <joint name="${prefix}joint3" type="revolute">
       <xacro:openarm-kinematics name="joint3" config="${kinematics}" />
@@ -54,5 +60,5 @@
       <xacro:openarm-limits name="joint4" config="${joint_limits}" />
     </joint>
-    <xacro:link_with_sc no_prefix="${no_prefix}" name="link5" gazebo="${gazebo}" kinematics_link="${kinematics_link}" />
+    <xacro:link_with_sc no_prefix="${no_prefix}" name="link5" gazebo="${gazebo}" kinematics_link="${kinematics_link}" reflect="${reflect}" />
     <joint name="${prefix}joint5" type="revolute">
       <xacro:openarm-kinematics name="joint5" config="${kinematics}" />
@@ -62,5 +68,5 @@
       <xacro:openarm-limits name="joint5" config="${joint_limits}" />
     </joint>
-    <xacro:link_with_sc no_prefix="${no_prefix}" name="link6" gazebo="${gazebo}" kinematics_link="${kinematics_link}"/>
+    <xacro:link_with_sc no_prefix="${no_prefix}" name="link6" gazebo="${gazebo}" kinematics_link="${kinematics_link}" reflect="${reflect}"/>
     <joint name="${prefix}joint6" type="revolute">
       <xacro:openarm-kinematics name="joint6" config="${kinematics}" />
@@ -70,5 +76,5 @@
       <xacro:openarm-limits name="joint6" config="${joint_limits}" />
     </joint>
-    <xacro:link_with_sc no_prefix="${no_prefix}" name="link7" gazebo="${gazebo}" rpy="0 0 0"  kinematics_link="${kinematics_link}"/>
+    <xacro:link_with_sc no_prefix="${no_prefix}" name="link7" gazebo="${gazebo}" rpy="0 0 0"  kinematics_link="${kinematics_link}" reflect="${reflect}"/>
     <joint name="${prefix}joint7" type="revolute">
       <xacro:openarm-kinematics name="joint7" config="${kinematics}" />

File: openarm_description/urdf/arm/openarm_macro.xacro (robot description, xacro)
@@ -32,5 +32,5 @@
   <!-- self_collision_geometries:  self <collision> models        -->
   <!-- ========================================================== -->
-  <xacro:macro name="link_with_sc" params="name no_prefix:='false' rpy:='0 0 0' gazebo:=false kinematics_link">
+  <xacro:macro name="link_with_sc" params="name no_prefix:='false' rpy:='0 0 0' gazebo:=false kinematics_link reflect:=1">
     <xacro:property name="prefix" value="${'' if no_prefix else arm_prefix + arm_type + '_'}" />
     <link name="${prefix}${name}">
@@ -38,5 +38,5 @@
         <xacro:openarm-kinematics-link config="${kinematics_link}" name="${name}" />
         <geometry>
-          <mesh filename="package://${description_pkg}/meshes/arm/${arm_type}/visual/${name}.dae" scale="0.001 0.001 0.001" />
+          <mesh filename="package://${description_pkg}/meshes/arm/${arm_type}/visual/${name}.dae" scale="0.001 ${0.001*reflect} 0.001" />
         </geometry>
       </visual>
@@ -44,5 +44,5 @@
         <xacro:openarm-kinematics-link config="${kinematics_link}" name="${name}" />
         <geometry>
-          <mesh filename="package://openarm_description/meshes/arm/${arm_type}/collision/${name}_symp.stl" scale="0.001 0.001 0.001" />
+          <mesh filename="package://openarm_description/meshes/arm/${arm_type}/collision/${name}_symp.stl" scale="0.001 ${0.001*reflect} 0.001" />
           <!-- <mesh filename="package://openarm_description/meshes/arm/${arm_type}/collision/${name}.stl" scale="0.001 0.001 0.001" /> -->
         </geometry>

File: openarm_description/urdf/ee/openarm_hand.xacro (robot description, xacro)
@@ -2,5 +2,5 @@
 <robot xmlns:xacro="http://www.ros.org/wiki/xacro" name="hand">
   <!-- safety_distance: Minimum safety distance in [m] by which the collision volumes are expanded and which is enforced during robot motions -->
-  <xacro:macro name="openarm_hand" params="connected_to:='' arm_type arm_prefix:='' ee_type ee_inertials rpy_ee:='0 0 0' xyz_ee:='0 0 0' tcp_xyz:='0 0 0.0' tcp_rpy:='0 0 0' gazebo:=false description_pkg:=openarm_description">
+  <xacro:macro name="openarm_hand" params="connected_to:='' arm_type arm_prefix:='' ee_type ee_inertials ee_kinematics_link rpy_ee:='0 0 0' xyz_ee:='0 0 0' tcp_xyz:='0 0 0.0' tcp_rpy:='0 0 0' gazebo:=false description_pkg:=openarm_description">
     <xacro:property name="ee_prefix" default=""/>
     <xacro:unless value="${arm_type == ''}">

File: openarm_description/urdf/ee/openarm_hand_macro.xacro (robot description, xacro)
@@ -48,3 +48,13 @@
     </link>
   </xacro:macro>
+  <xacro:macro name="openarm-ee-kinematics" params="config name">
+      <xacro:property name="kinematics" value="${config[name]['kinematic']}" lazy_eval="false" />
+      <origin rpy="${kinematics.roll} ${kinematics.pitch} ${kinematics.yaw}"
+            xyz="${kinematics.x} ${kinematics.y} ${kinematics.z}" />
+  </xacro:macro>
+  <xacro:macro name="openarm-ee-kinematics-link" params="config name">
+    <xacro:property name="kinematics_link" value="${config[name]['kinematic']}" lazy_eval="false" />
+    <origin rpy="${kinematics_link.roll} ${kinematics_link.pitch} ${kinematics_link.yaw}"
+            xyz="${kinematics_link.x} ${kinematics_link.y} ${kinematics_link.z}" />
+  </xacro:macro>
 </robot>

File: openarm_description/urdf/robot/openarm_robot.xacro (robot description, xacro)
@@ -11,4 +11,5 @@
             body_kinematics
             body_kinematics_link
+            ee_kinematics_link
             parent:='world'
             xyz:='0 0 0'
@@ -98,5 +99,5 @@
         <xacro:include filename="$(find openarm_description)/urdf/ee/openarm_hand.xacro"/>
         <xacro:include filename="$(find openarm_description)/urdf/ee/openarm_hand_macro.xacro" />
-        <xacro:include filename="$(find openarm_description)/urdf/${ee_type}_arguments.xacro" />
+        <xacro:include filename="$(find openarm_description)/urdf/ee/${ee_type}_arguments.xacro" />
         <xacro:property name="special_connection" value="$(arg special_connection)" />
         <xacro:property name="connection" value="${special_connection if special_connection != '' else arm_type + '_link8'}" />
@@ -106,4 +107,5 @@
             arm_prefix="${arm_prefix_modified}"
             ee_type="${ee_type}"
+            ee_kinematics_link="${xacro.load_yaml('$(find openarm_description)/config/hand/openarm_hand/kinematics_link.yaml')}"
             ee_inertials="${xacro.load_yaml('$(find openarm_description)/config/hand/$(arg ee_type)/hand_inertials.yaml')}"
             rpy_ee="$(arg rpy_ee)"
@@ -118,5 +120,5 @@
         <xacro:include filename="$(find openarm_description)/urdf/ee/ee_with_one_link.xacro"/>
         <xacro:include filename="$(find openarm_description)/urdf/ee/openarm_hand_macro.xacro" />
-        <xacro:include filename="$(find openarm_description)/urdf/${ee_type}_arguments.xacro" />
+        <xacro:include filename="$(find openarm_description)/urdf/ee/${ee_type}_arguments.xacro" />
         <xacro:property name="special_connection" value="$(arg special_connection)" />
         <xacro:property name="connection" value="${special_connection if special_connection == '' else arm_type + '_link8'}" />
@@ -127,4 +129,5 @@
             ee_type="${ee_type}"
             ee_inertials="${xacro.load_yaml('$(find openarm_description)/config/hand/$(arg ee_type)_inertials.yaml')}"
+            ee_kinematics_link="${xacro.load_yaml('$(find openarm_description)/config/hand/openarm_hand/kinematics_link.yaml')}"
             rpy_ee="$(arg rpy_ee)"
             xyz_ee="$(arg xyz_ee)"

File: openarm_description/urdf/robot/v10.urdf.xacro (robot description, xacro)
@@ -12,5 +12,5 @@
   <xacro:arg name="no_prefix" default="false"/>
   <!-- Should an end-effector be mounted at the flange?" -->
-  <xacro:arg name="hand" default="false" />
+  <xacro:arg name="hand" default="true" />
   <!-- Which end-effector would be mounted at the flange?" -->
   <xacro:arg name="ee_type" default="openarm_hand" />
@@ -34,5 +34,6 @@
   <xacro:arg name="gazebo_effort" default="false" />
   <!-- For a multi arm setup, we need a threaded robot running async-->
-  <xacro:arg name="bimanual" default="true" />
+  <xacro:arg name="bimanual" default="false" />
+  <!-- used in bimanual -->
   <xacro:arg name="right_arm_base_xyz" default="0.0 0.07 0.83" />
   <xacro:arg name="right_arm_base_rpy" default="-1.5708 0 0" />
@@ -49,4 +50,5 @@
   body_kinematics="${xacro.load_yaml('$(find openarm_description)/config/body/v10/kinematics.yaml')}"
   body_kinematics_link="${xacro.load_yaml('$(find openarm_description)/config/body/v10/kinematics.yaml')}"
+  ee_kinematics_link="${xacro.load_yaml('$(find openarm_description)/config/hand/openarm_hand/kinematics_link.yaml')}"
   gazebo="$(arg gazebo)"
   hand="$(arg hand)"
@@ -64,5 +66,5 @@
   bimanual="$(arg bimanual)"
   right_arm_base_xyz="$(arg right_arm_base_xyz)"
-  left_arm_base_xyz="$(arg left_arm_base_rpy)"
+  left_arm_base_xyz="$(arg left_arm_base_xyz)"
   right_arm_base_rpy="$(arg right_arm_base_rpy)"
   left_arm_base_rpy="$(arg left_arm_base_rpy)"

Commit message: fix: right left inversion of order

File: openarm_description/urdf/arm/openarm_arm.xacro (robot description, xacro)
@@ -6,5 +6,5 @@
   <!-- kinematics: description of the kinematics that comes from a YAML file. Example definition: ${xacro.load_yaml('$(find openarm_description)/robots/fr3/kinematics.yaml')} -->
   <!-- inertials: description of the inertials that comes from a YAML file. Example definition: ${xacro.load_yaml('$(find openarm_description)/robots/fr3/inertials.yaml')} -->
-  <xacro:macro name="openarm_arm" params="arm_type arm_prefix:='' no_prefix:=false description_pkg:='openarm_description' connected_to:='base' xyz:='0 0 0' rpy:='0 0 0' gazebo:='false' joint_limits inertials kinematics kinematics_link" >
+  <xacro:macro name="openarm_arm" params="arm_type arm_prefix:='' no_prefix:=false description_pkg:='openarm_description' connected_to:='base' xyz:='0 0 0' rpy:='0 0 0' gazebo:='false' joint_limits inertials kinematics kinematics_link kinematics_offset:=none " >
     <!-- Define a property that defaults to 'arm_prefix_arm_type' concatenated with an underscore if 'no_prefix' is not set -->
     <xacro:property name="prefix" value="${'' if no_prefix else arm_prefix + arm_type + '_'}" />
@@ -38,5 +38,5 @@
     <xacro:link_with_sc no_prefix="${no_prefix}" name="link2" gazebo="${gazebo}" kinematics_link="${kinematics_link}" reflect="${reflect}"/>
     <joint name="${prefix}joint2" type="revolute">
-      <xacro:openarm-kinematics name="joint2" config="${kinematics}" />
+      <xacro:openarm-kinematics name="joint2" config="${kinematics}" offset="${kinematics_offset}" />
       <parent link="${prefix}link1" />
       <child link="${prefix}link2" />

File: openarm_description/urdf/arm/openarm_macro.xacro (robot description, xacro)
@@ -32,5 +32,5 @@
   <!-- self_collision_geometries:  self <collision> models        -->
   <!-- ========================================================== -->
-  <xacro:macro name="link_with_sc" params="name no_prefix:='false' rpy:='0 0 0' gazebo:=false kinematics_link reflect:=1">
+  <xacro:macro name="link_with_sc" params="name no_prefix:='false' rpy:='0 0 0' gazebo:=false kinematics_link:=''  reflect:=1">
     <xacro:property name="prefix" value="${'' if no_prefix else arm_prefix + arm_type + '_'}" />
     <link name="${prefix}${name}">
@@ -177,8 +177,17 @@
   <!-- name   - Name of the joint for which to add kinematics to                 -->
   <!-- ========================================================================= -->
-  <xacro:macro name="openarm-kinematics" params="config name">
-      <xacro:property name="kinematics" value="${config[name]['kinematic']}" lazy_eval="false" />
-      <origin rpy="${kinematics.roll} ${kinematics.pitch} ${kinematics.yaw}"
-             xyz="${kinematics.x} ${kinematics.y} ${kinematics.z}" />
+  <xacro:macro name="openarm-kinematics" params="name config offset:=none">
+    <xacro:property name="kinematics" value="${config[name]['kinematic']}" lazy_eval="false" />
+    <xacro:if value="${offset != 'none'}">
+      <xacro:property name="offset" value="${offset[name]['kinematic_offset']}" lazy_eval="false" />
+      <origin
+        xyz="${kinematics.x + offset.x} ${kinematics.y + offset.y} ${kinematics.z + offset.z}"
+        rpy="${kinematics.roll + offset.roll} ${kinematics.pitch + offset.pitch} ${kinematics.yaw + offset.yaw}" />
+    </xacro:if>
+    <xacro:unless value="${offset != 'none'}">
+      <origin
+        xyz="${kinematics.x} ${kinematics.y} ${kinematics.z}"
+        rpy="${kinematics.roll} ${kinematics.pitch} ${kinematics.yaw}" />
+    </xacro:unless>
   </xacro:macro>
   <xacro:macro name="openarm-kinematics-link" params="config name">

File: openarm_description/urdf/robot/openarm_robot.xacro (robot description, xacro)
@@ -6,4 +6,5 @@
             kinematics
             kinematics_link
+            kinematics_offset
             inertials
             body_type
@@ -74,5 +75,6 @@
         inertials="${inertials}"
         kinematics="${kinematics}"
-        kinematics_link="${kinematics_link}" />
+        kinematics_link="${kinematics_link}"
+        kinematics_offset="${kinematics_offset}" />
         <xacro:openarm_arm_ros2_control
         arm_type="${arm_type}"
@@ -99,5 +101,6 @@
         inertials="${inertials}"
         kinematics="${kinematics}"
-        kinematics_link="${kinematics_link}" />
+        kinematics_link="${kinematics_link}"
+        kinematics_offset="${kinematics_offset}" />
         <xacro:openarm_arm_ros2_control
         arm_type="${arm_type}"
@@ -110,5 +113,5 @@
         hand="${hand}"
         bimanual="true"
-      />
+        />
         <xacro:if value="${hand and ee_type == 'openarm_hand'}">
             <xacro:openarm_hand
@@ -214,6 +217,6 @@
             <child  link="${arm_type}_link0" />
             </joint>
-        </xacro:if>
-        <xacro:gazebo-joint joint="${arm_type}_joint1" transmission="hardware_interface/PositionJointInterface" />
+        </xacro:if> -->
+        <!-- <xacro:gazebo-joint joint="${arm_type}_joint1" transmission="hardware_interface/PositionJointInterface" />
         <xacro:gazebo-joint joint="${arm_type}_joint2" transmission="hardware_interface/PositionJointInterface" />
         <xacro:gazebo-joint joint="${arm_type}_joint3" transmission="hardware_interface/PositionJointInterface" />
@@ -235,11 +238,11 @@
         <xacro:gazebo-joint joint="${arm_type}_joint5" transmission="hardware_interface/EffortJointInterface" />
         <xacro:gazebo-joint joint="${arm_type}_joint6" transmission="hardware_interface/EffortJointInterface" />
-        <xacro:gazebo-joint joint="${arm_type}_joint7" transmission="hardware_interface/EffortJointInterface" />
-        <xacro:transmission-openarm-state arm_type="${arm_type}" />
+        <xacro:gazebo-joint joint="${arm_type}_joint7" transmission="hardware_interface/EffortJointInterface" />  -->
+        <!-- <xacro:transmission-openarm-state arm_type="${arm_type}" />
         <xacro:transmission-openarm-model arm_type="${arm_type}"
             root="${arm_type}_joint1"
             tip="${arm_type}_joint8"
-        />
-        <xacro:if value="${ee_type == 'openarm_hand'}">
+        /> -->
+        <!-- <xacro:if value="${ee_type == 'openarm_hand'}">
             <xacro:gazebo-joint joint="${arm_type}_finger_joint1" transmission="hardware_interface/EffortJointInterface" />
             <xacro:gazebo-joint joint="${arm_type}_finger_joint2" transmission="hardware_interface/EffortJointInterface" />
@@ -247,18 +250,4 @@
             <xacro:gazebo-friction link="${arm_type}_rightfinger" mu="1.13" />
         </xacro:if>
-        </xacro:if>
-        <xacro:if value="${ros2_control}">
-        <xacro:include filename="$(find openarm_description)/urdf/ros2_control/openarm_arm.ros2_control.xacro"/>
-        <xacro:openarm_arm_ros2_control
-            arm_type="${arm_type}"
-            can="${can}"
-            use_fake_hardware="$(arg use_fake_hardware)"
-            fake_sensor_commands="$(arg fake_sensor_commands)"
-            gazebo="$(arg gazebo)"
-            hand="$(arg hand)"
-            gazebo_effort="$(arg gazebo_effort)"
-            arm_prefix="${arm_prefix}"
-            multi_arm="$(arg multi_arm)"
-        />
         </xacro:if> -->
   </xacro:macro>

File: openarm_description/urdf/robot/v10.urdf.xacro (robot description, xacro)
@@ -35,8 +35,8 @@
   <xacro:arg name="bimanual" default="false" />
   <!-- used in bimanual -->
-  <xacro:arg name="right_arm_base_xyz" default="0.0 0.07 0.83" />
-  <xacro:arg name="right_arm_base_rpy" default="-1.5708 0 0" />
-  <xacro:arg name="left_arm_base_xyz" default="0.0 -0.07 0.83" />
-  <xacro:arg name="left_arm_base_rpy" default="1.5708 0 0" />
+  <xacro:arg name="right_arm_base_xyz" default="0.0 -0.07 0.83" />
+  <xacro:arg name="right_arm_base_rpy" default="1.5708 0 0" />
+  <xacro:arg name="left_arm_base_xyz" default="0.0 0.07 0.83" />
+  <xacro:arg name="left_arm_base_rpy" default="-1.5708 0 0" />
   <xacro:openarm_robot
   arm_type="v10"
@@ -46,4 +46,5 @@
   kinematics="${xacro.load_yaml('$(find openarm_description)/config/v10/kinematics.yaml')}"
   kinematics_link="${xacro.load_yaml('$(find openarm_description)/config/v10/kinematics_link.yaml')}"
+  kinematics_offset="${xacro.load_yaml('$(find openarm_description)/config/v10/kinematics_offset.yaml')}"
   body_inertials="${xacro.load_yaml('$(find openarm_description)/config/body/v10/inertials.yaml')}"
   body_kinematics="${xacro.load_yaml('$(find openarm_description)/config/body/v10/kinematics.yaml')}"
