Commit message: fix: joint2 angle limit

File: openarm_description/urdf/arm/openarm_arm.xacro (robot description, xacro)
@@ -10,8 +10,8 @@
     <xacro:property name="prefix" value="${'' if no_prefix else arm_prefix + arm_type + '_'}" />
     <xacro:if value="${arm_prefix == 'right_'}">
-      <xacro:property name="reflect" value="-1" />
+      <xacro:property name="reflect" value="1" />
     </xacro:if>
     <xacro:unless value="${arm_prefix == 'right_'}">
-      <xacro:property name="reflect" value="1" />
+      <xacro:property name="reflect" value="-1" />
     </xacro:unless>
     <xacro:if value="${gazebo}">
@@ -30,5 +30,5 @@
     <xacro:link_with_sc no_prefix="${no_prefix}" name="link1" gazebo="${gazebo}" kinematics_link="${kinematics_link}" reflect="${reflect}"/>
     <joint name="${prefix}joint1" type="revolute">
-      <xacro:openarm-kinematics name="joint1" config="${kinematics}" />
+      <xacro:openarm-kinematics name="joint1" config="${kinematics}" reflect="${reflect}"/>
       <parent link="${prefix}link0" />
       <child link="${prefix}link1" />
@@ -37,10 +37,16 @@
     </joint>
     <xacro:link_with_sc no_prefix="${no_prefix}" name="link2" gazebo="${gazebo}" kinematics_link="${kinematics_link}" reflect="${reflect}"/>
+    <xacro:if value="${prefix.find('right_') != -1}">
+      <xacro:property name="limit_offset_joint2" value="${pi/2}" />
+    </xacro:if>
+    <xacro:if value="${prefix.find('left_') != -1}">
+      <xacro:property name="limit_offset_joint2" value="${-pi/2}" />
+    </xacro:if>
     <joint name="${prefix}joint2" type="revolute">
-      <xacro:openarm-kinematics name="joint2" config="${kinematics}" offset="${kinematics_offset}" />
+      <xacro:openarm-kinematics name="joint2" config="${kinematics}" offset="${kinematics_offset}" reflect="${reflect}"/>
       <parent link="${prefix}link1" />
       <child link="${prefix}link2" />
       <axis xyz="-1 0 0" />
-      <xacro:openarm-limits name="joint2" config="${joint_limits}" />
+      <xacro:openarm-limits name="joint2" config="${joint_limits}" reflect="${reflect}" offset="${limit_offset_joint2}"/>
     </joint>
     <xacro:link_with_sc no_prefix="${no_prefix}" name="link3" gazebo="${gazebo}" kinematics_link="${kinematics_link}" reflect="${reflect}"/>

File: openarm_description/urdf/arm/openarm_macro.xacro (robot description, xacro)
@@ -160,14 +160,23 @@
   <!-- name   - Name of the joint for which to add limits to                     -->
   <!-- ========================================================================= -->
-  <xacro:macro name="openarm-limits" params="config name">
-      <xacro:property name="limits" value="${config[name]['limit']}" lazy_eval="false" />
-      <limit lower="${limits.lower}"
-             upper="${limits.upper}"
-             effort="${limits.effort}"
-             velocity="${limits.velocity}" />
-      <!-- <safety_controller k_position="100.0"
-                         k_velocity="40.0"
-                         soft_lower_limit="${limits.lower}"
-                         soft_upper_limit="${limits.upper}" /> -->
+  <xacro:macro name="openarm-limits" params="name config reflect:=1 offset:=0">
+    <xacro:property name="limits" value="${config[name]['limit']}" lazy_eval="false"/>
+    <xacro:property name="raw_lower" value="${limits.lower * reflect + offset}" />
+    <xacro:property name="raw_upper" value="${limits.upper * reflect + offset}" />
+    <xacro:property name="lower" value="0.0" />
+    <xacro:property name="upper" value="0.0" />
+    <xacro:if value="${raw_lower &lt; raw_upper}">
+      <xacro:property name="lower" value="${raw_lower}" />
+      <xacro:property name="upper" value="${raw_upper}" />
+    </xacro:if>
+    <xacro:unless value="${raw_lower &lt; raw_upper}">
+      <xacro:property name="lower" value="${raw_upper}" />
+      <xacro:property name="upper" value="${raw_lower}" />
+    </xacro:unless>
+    <limit
+      lower="${lower}"
+      upper="${upper}"
+      effort="${limits.effort}"
+      velocity="${limits.velocity}" />
   </xacro:macro>
   <!-- ========================================================================= -->
@@ -177,5 +186,5 @@
   <!-- name   - Name of the joint for which to add kinematics to                 -->
   <!-- ========================================================================= -->
-  <xacro:macro name="openarm-kinematics" params="name config offset:=none">
+  <xacro:macro name="openarm-kinematics" params="name config offset:=none reflect:=1">
     <xacro:property name="kinematics" value="${config[name]['kinematic']}" lazy_eval="false" />
     <xacro:if value="${offset != 'none'}">
@@ -183,5 +192,5 @@
       <origin
         xyz="${kinematics.x + offset.x} ${kinematics.y + offset.y} ${kinematics.z + offset.z}"
-        rpy="${kinematics.roll + offset.roll} ${kinematics.pitch + offset.pitch} ${kinematics.yaw + offset.yaw}" />
+        rpy="${kinematics.roll + reflect*offset.roll} ${kinematics.pitch +  reflect*offset.pitch} ${kinematics.yaw +  reflect*offset.yaw}" />
     </xacro:if>
     <xacro:unless value="${offset != 'none'}">

Commit message: fix: undefined property

File: openarm_description/urdf/arm/openarm_arm.xacro (robot description, xacro)
@@ -36,5 +36,7 @@
       <xacro:openarm-limits name="joint1" config="${joint_limits}" />
     </joint>
+    <!-- for bimanual offset -->
     <xacro:link_with_sc no_prefix="${no_prefix}" name="link2" gazebo="${gazebo}" kinematics_link="${kinematics_link}" reflect="${reflect}"/>
+    <xacro:property name="limit_offset_joint2" value="0" />
     <xacro:if value="${prefix.find('right_') != -1}">
       <xacro:property name="limit_offset_joint2" value="${pi/2}" />

Commit message: fix: joint link name and gripper origiin

File: openarm_description/urdf/arm/openarm_arm.xacro (robot description, xacro)
@@ -8,5 +8,6 @@
   <xacro:macro name="openarm_arm" params="arm_type arm_prefix:='' no_prefix:=false description_pkg:='openarm_description' connected_to:='base' xyz:='0 0 0' rpy:='0 0 0' gazebo:='false' joint_limits inertials kinematics kinematics_link kinematics_offset:=none " >
     <!-- Define a property that defaults to 'arm_prefix_arm_type' concatenated with an underscore if 'no_prefix' is not set -->
-    <xacro:property name="prefix" value="${'' if no_prefix else arm_prefix + arm_type + '_'}" />
+    <!-- <xacro:property name="prefix" value="${'' if no_prefix else arm_prefix + arm_type + '_'}" /> -->
+    <xacro:property name="prefix" value="${'' if no_prefix else arm_prefix + 'openarm' + '_'}" />
     <xacro:if value="${arm_prefix == 'right_'}">
       <xacro:property name="reflect" value="1" />

File: openarm_description/urdf/arm/openarm_macro.xacro (robot description, xacro)
@@ -7,18 +7,22 @@
   <!-- inertial: Dictionary of inertia properties (see inertial.yaml) -->
   <!-- ============================================================== -->
-  <xacro:macro name="openarm-inertials" params="name inertials:=^">
-      <xacro:unless value="${name in inertials}">${xacro.warning('No inertia properties defined for: ' + name)}</xacro:unless>
-      <xacro:if value="${name in inertials}">
-        <!-- Access inertia properties of link 'name' -->
-        <xacro:property name="link_inertials" value="${inertials[name]}" lazy_eval="false" />
-        <inertial>
-          <origin rpy="${link_inertials.origin.rpy}" xyz="${link_inertials.origin.xyz}" />
-          <mass value="${link_inertials.mass}" />
-          <xacro:if value="${'inertia' in link_inertials}">
-            <xacro:property name="I" value="${link_inertials.inertia}" />
-            <inertia ixx="${I.xx}" ixy="${I.xy}" ixz="${I.xz}" iyy="${I.yy}" iyz="${I.yz}" izz="${I.zz}" />
-          </xacro:if>
-        </inertial>
-      </xacro:if>
+  <xacro:macro name="openarm-inertials" params="name inertials:=^ reflect:=1">
+    <xacro:unless value="${name in inertials}">
+      ${xacro.warning('No inertia properties defined for: ' + name)}
+    </xacro:unless>
+    <xacro:if value="${name in inertials}">
+      <xacro:property name="I" value="${inertials[name]}" lazy_eval="false" />
+      <inertial>
+        <origin
+          xyz="${I.origin.x} ${reflect * I.origin.y} ${I.origin.z}"
+          rpy="${I.origin.roll} ${I.origin.pitch} ${I.origin.yaw}" />
+        <mass value="${I.mass}" />
+        <xacro:if value="${'inertia' in I}">
+          <xacro:property name="inert" value="${I.inertia}" />
+          <inertia ixx="${inert.xx}" ixy="${inert.xy}" ixz="${inert.xz}"
+                   iyy="${inert.yy}" iyz="${inert.yz}" izz="${inert.zz}" />
+        </xacro:if>
+      </inertial>
+    </xacro:if>
   </xacro:macro>
   <!-- ========================================================== -->
@@ -33,5 +37,6 @@
   <!-- ========================================================== -->
   <xacro:macro name="link_with_sc" params="name no_prefix:='false' rpy:='0 0 0' gazebo:=false kinematics_link:=''  reflect:=1">
-    <xacro:property name="prefix" value="${'' if no_prefix else arm_prefix + arm_type + '_'}" />
+    <!-- <xacro:property name="prefix" value="${'' if no_prefix else arm_prefix + arm_type + '_'}" /> -->
+    <xacro:property name="prefix" value="${'' if no_prefix else arm_prefix + 'openarm' + '_'}" />
     <link name="${prefix}${name}">
       <visual name="${prefix}${name}_visual">
@@ -161,5 +166,5 @@
   <!-- ========================================================================= -->
   <xacro:macro name="openarm-limits" params="name config reflect:=1 offset:=0">
-    <xacro:property name="limits" value="${config[name]['limit']}" lazy_eval="false"/>
+    <xacro:property name="limits" value="${config[name]['limit']}"/>
     <xacro:property name="raw_lower" value="${limits.lower * reflect + offset}" />
     <xacro:property name="raw_upper" value="${limits.upper * reflect + offset}" />
@@ -192,10 +197,10 @@
       <origin
         xyz="${kinematics.x + offset.x} ${kinematics.y + offset.y} ${kinematics.z + offset.z}"
-        rpy="${kinematics.roll + reflect*offset.roll} ${kinematics.pitch +  reflect*offset.pitch} ${kinematics.yaw +  reflect*offset.yaw}" />
+        rpy="${reflect*(kinematics.roll + offset.roll)} ${reflect*(kinematics.pitch + offset.pitch)} ${reflect*(kinematics.yaw + offset.yaw)}" />
     </xacro:if>
     <xacro:unless value="${offset != 'none'}">
       <origin
         xyz="${kinematics.x} ${kinematics.y} ${kinematics.z}"
-        rpy="${kinematics.roll} ${kinematics.pitch} ${kinematics.yaw}" />
+        rpy="${reflect*kinematics.roll} ${reflect*kinematics.pitch} ${reflect*kinematics.yaw}" />
     </xacro:unless>
   </xacro:macro>

File: openarm_description/urdf/ee/openarm_hand.xacro (robot description, xacro)
@@ -2,11 +2,13 @@
 <robot xmlns:xacro="http://www.ros.org/wiki/xacro" name="hand">
   <!-- safety_distance: Minimum safety distance in [m] by which the collision volumes are expanded and which is enforced during robot motions -->
-  <xacro:macro name="openarm_hand" params="connected_to:='' arm_type arm_prefix:='' ee_type ee_inertials ee_kinematics_link rpy_ee:='0 0 0' xyz_ee:='0 0 0' tcp_xyz:='0 0.1 0' tcp_rpy:='0 0 0' gazebo:=false description_pkg:=openarm_description">
+  <xacro:macro name="openarm_hand" params="connected_to:='' arm_type arm_prefix:='' ee_type ee_inertials ee_kinematics_link rpy_ee:='0 0 0' xyz_ee:='0 0 0' tcp_xyz:='0 0 0' tcp_rpy:='0 0 0' gazebo:=false description_pkg:=openarm_description">
     <xacro:property name="ee_prefix" default=""/>
     <xacro:unless value="${arm_type == ''}">
-      <xacro:property name="ee_prefix" value="${arm_prefix}${arm_type}_" />
+      <!-- <xacro:property name="ee_prefix" value="${arm_prefix}${arm_type}_" /> -->
+      <xacro:property name="ee_prefix" value="${arm_prefix}openarm_" />
     </xacro:unless>
     <xacro:unless value="${connected_to == ''}">
-      <joint name="${ee_prefix}hand_joint" type="fixed">
+      <!-- <joint name="${ee_prefix}hand_joint" type="fixed"> -->
+      <joint name="openarm_hand_joint" type="fixed">
         <parent link="${connected_to}" />
         <child link="${ee_prefix}hand" />
@@ -19,17 +21,18 @@
     <link name="${ee_prefix}hand_tcp" />
     <joint name="${ee_prefix}hand_tcp_joint" type="fixed">
-      <origin xyz="${tcp_xyz}" rpy="${tcp_rpy}" />
+      <origin xyz="0 0.1 0.06" rpy="${tcp_rpy}" />
+      <!-- <origin xyz="${tcp_xyz}" rpy="${tcp_rpy}" /> -->
       <parent link="${ee_prefix}hand" />
       <child link="${ee_prefix}hand_tcp" />
     </joint>
-    <link name="${ee_prefix}leftfinger">
-      <visual name="${ee_prefix}leftfinger_visual">
-        <xacro:openarm-ee-kinematics-link config="${ee_kinematics_link}" name="leftfinger" />
+    <link name="${ee_prefix}left_finger">
+      <visual name="${ee_prefix}left_finger_visual">
+        <xacro:openarm-ee-kinematics-link config="${ee_kinematics_link}" name="left_finger" />
         <geometry>
           <mesh filename="package://${description_pkg}/meshes/ee/${ee_type}/visual/finger.dae" scale="0.001 0.001 0.001"/>
         </geometry>
       </visual>
-      <collision name="${ee_prefix}leftfinger_collision">
-        <xacro:openarm-ee-kinematics-link config="${ee_kinematics_link}" name="leftfinger" />
+      <collision name="${ee_prefix}left_finger_collision">
+        <xacro:openarm-ee-kinematics-link config="${ee_kinematics_link}" name="left_finger" />
         <geometry>
           <mesh filename="package://${description_pkg}/meshes/ee/${ee_type}/collision/finger.stl" scale="0.001 0.001 0.001" />
@@ -37,16 +40,16 @@
       </collision>
       <xacro:if value="${gazebo}">
-        <xacro:ee-inertials name="leftfinger" />
+        <xacro:ee-inertials name="left_finger" />
       </xacro:if>
     </link>
-    <link name="${ee_prefix}rightfinger">
-      <visual name="${ee_prefix}rightfinger_visual">
-        <xacro:openarm-ee-kinematics-link config="${ee_kinematics_link}" name="rightfinger" />
+    <link name="${ee_prefix}right_finger">
+      <visual name="${ee_prefix}right_finger_visual">
+        <xacro:openarm-ee-kinematics-link config="${ee_kinematics_link}" name="right_finger" />
         <geometry>
           <mesh filename="package://${description_pkg}/meshes/ee/${ee_type}/visual/finger.dae" scale="0.001 -0.001 0.001"/>
         </geometry>
       </visual>
-      <collision name="${ee_prefix}rightfinger_collision">
-        <xacro:openarm-ee-kinematics-link config="${ee_kinematics_link}" name="leftfinger" />
+      <collision name="${ee_prefix}right_finger_collision">
+        <xacro:openarm-ee-kinematics-link config="${ee_kinematics_link}" name="left_finger" />
         <geometry>
           <mesh filename="package://${description_pkg}/meshes/ee/${ee_type}/collision/finger.stl" scale="0.001 -0.001 0.001" />
@@ -54,11 +57,11 @@
       </collision>
       <xacro:if value="${gazebo}">
-        <xacro:ee-inertials name="rightfinger" />
+        <xacro:ee-inertials name="right_finger" />
       </xacro:if>
     </link>
-    <joint name="${ee_prefix}finger_joint1" type="prismatic">
+    <!-- <joint name="${ee_prefix}finger_joint1" type="prismatic">
       <parent link="${ee_prefix}hand" />
-      <child link="${ee_prefix}leftfinger" />
-      <origin xyz="0 0 0" rpy="0 0 0" />
+      <child link="${ee_prefix}right_finger" />
+      <origin xyz="0 0.05 0" rpy="0 0 0" />
       <axis xyz="0 -1 0" />
       <limit effort="100" lower="0.0" upper="0.044" velocity="0.2" />
@@ -66,6 +69,21 @@
     <joint name="${ee_prefix}finger_joint2" type="prismatic">
       <parent link="${ee_prefix}hand" />
-      <child link="${ee_prefix}rightfinger" />
-      <origin xyz="0 0 0" rpy="0 0 0" />
+      <child link="${ee_prefix}left_finger" />
+      <origin xyz="0 0.15 0" rpy="0 0 0" />
+      <axis xyz="0 1 0" />
+      <limit effort="100" lower="0.0" upper="0.044" velocity="0.2" />
+      <mimic joint="${ee_prefix}finger_joint1" />
+    </joint> -->
+    <joint name="${ee_prefix}finger_joint1" type="prismatic">
+      <parent link="${ee_prefix}hand" />
+      <child link="${ee_prefix}right_finger" />
+      <origin xyz="0 0.095 0" rpy="0 0 0" />
+      <axis xyz="0 -1 0" />
+      <limit effort="100" lower="0.0" upper="0.044" velocity="0.2" />
+    </joint>
+    <joint name="${ee_prefix}finger_joint2" type="prismatic">
+      <parent link="${ee_prefix}hand" />
+      <child link="${ee_prefix}left_finger" />
+      <origin xyz="0 0.105 0" rpy="0 0 0" />
       <axis xyz="0 1 0" />
       <limit effort="100" lower="0.0" upper="0.044" velocity="0.2" />

File: openarm_description/urdf/robot/openarm_robot.xacro (robot description, xacro)
@@ -172,5 +172,6 @@
         <xacro:if value="${hand and ee_type == 'openarm_hand'}">
         <xacro:property name="special_connection" value="$(arg special_connection)" />
-        <xacro:property name="connection" value="${special_connection if special_connection != '' else arm_type + '_link8'}" />
+        <!-- <xacro:property name="connection" value="${special_connection if special_connection != '' else arm_type + '_link8'}" /> -->
+        <xacro:property name="connection" value="${special_connection if special_connection != '' else 'openarm' + '_link8'}" />
         <xacro:openarm_hand
             connected_to="${arm_prefix_modified}${connection}"

File: openarm_description/urdf/robot/v10.urdf.xacro (robot description, xacro)
@@ -67,5 +67,5 @@
   xyz_ee='0 0 0'
   xyz_rpy='0 0 0'
-  tcp_xyz='0 0 0'
+  tcp_xyz='0 0.1 0.06'
   tcp_rpy='0 0 0'
   right_arm_base_xyz="$(arg right_arm_base_xyz)"

Commit message: fix: left right prefix position

File: openarm_description/urdf/arm/openarm_arm.xacro (robot description, xacro)
@@ -9,5 +9,6 @@
     <!-- Define a property that defaults to 'arm_prefix_arm_type' concatenated with an underscore if 'no_prefix' is not set -->
     <!-- <xacro:property name="prefix" value="${'' if no_prefix else arm_prefix + arm_type + '_'}" /> -->
-    <xacro:property name="prefix" value="${'' if no_prefix else arm_prefix + 'openarm' + '_'}" />
+    <!-- <xacro:property name="prefix" value="${'' if no_prefix else arm_prefix + 'openarm' + '_'}" /> -->
+    <xacro:property name="prefix" value="${'' if no_prefix else 'openarm' + '_' + arm_prefix}" />
     <xacro:if value="${arm_prefix == 'right_'}">
       <xacro:property name="reflect" value="1" />

File: openarm_description/urdf/arm/openarm_macro.xacro (robot description, xacro)
@@ -38,5 +38,5 @@
   <xacro:macro name="link_with_sc" params="name no_prefix:='false' rpy:='0 0 0' gazebo:=false kinematics_link:=''  reflect:=1">
     <!-- <xacro:property name="prefix" value="${'' if no_prefix else arm_prefix + arm_type + '_'}" /> -->
-    <xacro:property name="prefix" value="${'' if no_prefix else arm_prefix + 'openarm' + '_'}" />
+    <xacro:property name="prefix" value="${'' if no_prefix else 'openarm' + '_' +  arm_prefix}" />
     <link name="${prefix}${name}">
       <visual name="${prefix}${name}_visual">

File: openarm_description/urdf/ee/openarm_hand.xacro (robot description, xacro)
@@ -6,5 +6,5 @@
     <xacro:unless value="${arm_type == ''}">
       <!-- <xacro:property name="ee_prefix" value="${arm_prefix}${arm_type}_" /> -->
-      <xacro:property name="ee_prefix" value="${arm_prefix}openarm_" />
+      <xacro:property name="ee_prefix" value="openarm_${arm_prefix}" />
     </xacro:unless>
     <xacro:unless value="${connected_to == ''}">

File: openarm_description/urdf/robot/openarm_robot.xacro (robot description, xacro)
@@ -119,5 +119,5 @@
         <xacro:if value="${hand and ee_type == 'openarm_hand'}">
             <xacro:openarm_hand
-                connected_to="left_openarm_link8"
+                connected_to="openarm_left_link8"
                 arm_type="${arm_type}"
                 arm_prefix="left_"
@@ -133,5 +133,5 @@
             />
             <xacro:openarm_hand
-                connected_to="right_openarm_link8"
+                connected_to="openarm_right_link8"
                 arm_type="${arm_type}"
                 arm_prefix="right_"

File: openarm_description/urdf/robot/v10.urdf (robot description, URDF)
Before this commit: robot openarm, 13 links, 12 joints
Joints:
- joint openarm_hand_tcp_joint: origin xyz=0 0 0.0 rpy=0 0 0 -> xyz=0 0.1 0.06 rpy=0 0 0
