Commit message: delete: gazebo setting

File: openarm_description/urdf/arm/openarm_arm.xacro (robot description, xacro)
@@ -6,5 +6,5 @@
   <!-- kinematics: description of the kinematics that comes from a YAML file. Example definition: ${xacro.load_yaml('$(find openarm_description)/robots/fr3/kinematics.yaml')} -->
   <!-- inertials: description of the inertials that comes from a YAML file. Example definition: ${xacro.load_yaml('$(find openarm_description)/robots/fr3/inertials.yaml')} -->
-  <xacro:macro name="openarm_arm" params="arm_type arm_prefix:='' no_prefix:=false description_pkg:='openarm_description' connected_to:='base' xyz:='0 0 0' rpy:='0 0 0' gazebo:='false' joint_limits inertials kinematics kinematics_link kinematics_offset:=none " >
+  <xacro:macro name="openarm_arm" params="arm_type arm_prefix:='' no_prefix:=false description_pkg:='openarm_description' connected_to:='base' xyz:='0 0 0' rpy:='0 0 0' joint_limits inertials kinematics kinematics_link kinematics_offset:=none " >
     <!-- Define a property that defaults to 'arm_prefix_arm_type' concatenated with an underscore if 'no_prefix' is not set -->
     <!-- <xacro:property name="prefix" value="${'' if no_prefix else arm_prefix + arm_type + '_'}" /> -->
@@ -17,7 +17,7 @@
       <xacro:property name="reflect" value="-1" />
     </xacro:unless>
-    <xacro:if value="${gazebo}">
+    <!-- <xacro:if value="${gazebo}">
       <xacro:property name="connected_to" value="" />
-    </xacro:if>
+    </xacro:if> -->
     <xacro:unless value="${connected_to == ''}">
       <!-- <link name="${connected_to}">
@@ -29,6 +29,6 @@
       </joint>
     </xacro:unless>
-    <xacro:link_with_sc no_prefix="${no_prefix}" name="link0" gazebo="${gazebo}" kinematics_link="${kinematics_link}" reflect="${reflect}"/>
-    <xacro:link_with_sc no_prefix="${no_prefix}" name="link1" gazebo="${gazebo}" kinematics_link="${kinematics_link}" reflect="${reflect}"/>
+    <xacro:link_with_sc no_prefix="${no_prefix}" name="link0" kinematics_link="${kinematics_link}" reflect="${reflect}"/>
+    <xacro:link_with_sc no_prefix="${no_prefix}" name="link1" kinematics_link="${kinematics_link}" reflect="${reflect}"/>
     <joint name="${prefix}joint1" type="revolute">
       <xacro:openarm-kinematics name="joint1" config="${kinematics}" reflect="${reflect}"/>
@@ -39,5 +39,5 @@
     </joint>
     <!-- for bimanual offset -->
-    <xacro:link_with_sc no_prefix="${no_prefix}" name="link2" gazebo="${gazebo}" kinematics_link="${kinematics_link}" reflect="${reflect}"/>
+    <xacro:link_with_sc no_prefix="${no_prefix}" name="link2" kinematics_link="${kinematics_link}" reflect="${reflect}"/>
     <xacro:property name="limit_offset_joint2" value="0" />
     <xacro:if value="${prefix.find('right_') != -1}">
@@ -54,5 +54,5 @@
       <xacro:openarm-limits name="joint2" config="${joint_limits}" reflect="${reflect}" offset="${limit_offset_joint2}"/>
     </joint>
-    <xacro:link_with_sc no_prefix="${no_prefix}" name="link3" gazebo="${gazebo}" kinematics_link="${kinematics_link}" reflect="${reflect}"/>
+    <xacro:link_with_sc no_prefix="${no_prefix}" name="link3" kinematics_link="${kinematics_link}" reflect="${reflect}"/>
     <joint name="${prefix}joint3" type="revolute">
       <xacro:openarm-kinematics name="joint3" config="${kinematics}" />
@@ -62,5 +62,5 @@
       <xacro:openarm-limits name="joint3" config="${joint_limits}" />
     </joint>
-    <xacro:link_with_sc no_prefix="${no_prefix}" name="link4" gazebo="${gazebo}" kinematics_link="${kinematics_link}" />
+    <xacro:link_with_sc no_prefix="${no_prefix}" name="link4" kinematics_link="${kinematics_link}" />
     <joint name="${prefix}joint4" type="revolute">
       <xacro:openarm-kinematics name="joint4" config="${kinematics}" />
@@ -70,5 +70,5 @@
       <xacro:openarm-limits name="joint4" config="${joint_limits}" />
     </joint>
-    <xacro:link_with_sc no_prefix="${no_prefix}" name="link5" gazebo="${gazebo}" kinematics_link="${kinematics_link}" reflect="${reflect}" />
+    <xacro:link_with_sc no_prefix="${no_prefix}" name="link5" kinematics_link="${kinematics_link}" reflect="${reflect}" />
     <joint name="${prefix}joint5" type="revolute">
       <xacro:openarm-kinematics name="joint5" config="${kinematics}" />
@@ -78,5 +78,5 @@
       <xacro:openarm-limits name="joint5" config="${joint_limits}" />
     </joint>
-    <xacro:link_with_sc no_prefix="${no_prefix}" name="link6" gazebo="${gazebo}" kinematics_link="${kinematics_link}" reflect="${reflect}"/>
+    <xacro:link_with_sc no_prefix="${no_prefix}" name="link6" kinematics_link="${kinematics_link}" reflect="${reflect}"/>
     <joint name="${prefix}joint6" type="revolute">
       <xacro:openarm-kinematics name="joint6" config="${kinematics}" />
@@ -86,5 +86,5 @@
       <xacro:openarm-limits name="joint6" config="${joint_limits}" />
     </joint>
-    <xacro:link_with_sc no_prefix="${no_prefix}" name="link7" gazebo="${gazebo}" rpy="0 0 0"  kinematics_link="${kinematics_link}" reflect="${reflect}"/>
+    <xacro:link_with_sc no_prefix="${no_prefix}" name="link7" rpy="0 0 0"  kinematics_link="${kinematics_link}" reflect="${reflect}"/>
     <joint name="${prefix}joint7" type="revolute">
       <xacro:openarm-kinematics name="joint7" config="${kinematics}" />

File: openarm_description/urdf/arm/openarm_macro.xacro (robot description, xacro)
@@ -36,5 +36,5 @@
   <!-- self_collision_geometries:  self <collision> models        -->
   <!-- ========================================================== -->
-  <xacro:macro name="link_with_sc" params="name no_prefix:='false' rpy:='0 0 0' gazebo:=false kinematics_link:=''  reflect:=1">
+  <xacro:macro name="link_with_sc" params="name no_prefix:='false' rpy:='0 0 0' kinematics_link:=''  reflect:=1">
     <!-- <xacro:property name="prefix" value="${'' if no_prefix else arm_prefix + arm_type + '_'}" /> -->
     <xacro:property name="prefix" value="${'' if no_prefix else 'openarm' + '_' +  arm_prefix}" />
@@ -62,7 +62,6 @@
   <!-- transmission - type of the transmission of the joint       -->
   <!-- ========================================================== -->
-  <xacro:macro name="gazebo-joint" params="joint transmission:=hardware_interface/EffortJointInterface">
+  <!-- <xacro:macro name="gazebo-joint" params="joint transmission:=hardware_interface/EffortJointInterface">
     <gazebo reference="${joint}">
-      <!-- Needed for ODE to output external wrenches on joints -->
       <provideFeedback>true</provideFeedback>
     </gazebo>
@@ -76,6 +75,6 @@
       </actuator>
     </transmission>
-  </xacro:macro>
-  <xacro:macro name="gazebo-friction" params="link mu">
+  </xacro:macro> -->
+  <!-- <xacro:macro name="gazebo-friction" params="link mu">
     <gazebo reference="${link}">
       <collision>
@@ -84,7 +83,4 @@
           <contact>
             <ode>
-              <!-- These two parameter need application specific tuning. -->
-              <!-- Usually you want no "snap out" velocity and a generous -->
-              <!-- penetration depth to keep the grasping stable -->
               <max_vel>0</max_vel>
               <min_depth>0.001</min_depth>
@@ -101,5 +97,5 @@
       </collision>
     </gazebo>
-  </xacro:macro>
+  </xacro:macro> -->
   <!-- ========================================================== -->
   <!-- Adds the required tags to provide a `openarmStateInterface` -->

File: openarm_description/urdf/body/openarm_body.xacro (robot description, xacro)
@@ -10,5 +10,4 @@
               xyz:='0 0 0'
               rpy:='0 0 0'
-              gazebo:='false'
               inertials
               kinematics
@@ -26,5 +25,4 @@
     name="body_link0"
     no_prefix="${no_prefix}"
-    gazebo="${gazebo}"
     kinematics_link="${kinematics_link}" />
     </xacro:macro>

File: openarm_description/urdf/body/openarm_body_macro.xacro (robot description, xacro)
@@ -26,5 +26,4 @@
   <!--  * detailed meshes for environmental collision checking    -->
   <!--  * and coarse geometry models for self-collision checking  -->
-  <!--    (only if 'gazebo' param is set)                         -->
   <!--                                                            -->
   <!-- name:  Name of the robot link (without prefix)             -->
@@ -32,5 +31,5 @@
   <!-- self_collision_geometries:  self <collision> models        -->
   <!-- ========================================================== -->
-  <xacro:macro name="body_link_with_sc" params="name no_prefix:='false' rpy:='0 0 0' gazebo:=false kinematics_link">
+  <xacro:macro name="body_link_with_sc" params="name no_prefix:='false' rpy:='0 0 0' kinematics_link">
     <xacro:property name="prefix" value="${'' if no_prefix else body_prefix + body_type + '_'}" />
     <link name="${prefix}${name}">

File: openarm_description/urdf/ee/openarm_hand.xacro (robot description, xacro)
@@ -2,5 +2,5 @@
 <robot xmlns:xacro="http://www.ros.org/wiki/xacro" name="hand">
   <!-- safety_distance: Minimum safety distance in [m] by which the collision volumes are expanded and which is enforced during robot motions -->
-  <xacro:macro name="openarm_hand" params="connected_to:='' arm_type arm_prefix:='' ee_type ee_inertials ee_kinematics_link rpy_ee:='0 0 0' xyz_ee:='0 0 0' tcp_xyz:='0 0 0' tcp_rpy:='0 0 0' gazebo:=false description_pkg:=openarm_description">
+  <xacro:macro name="openarm_hand" params="connected_to:='' arm_type arm_prefix:='' ee_type ee_inertials ee_kinematics_link rpy_ee:='0 0 0' xyz_ee:='0 0 0' tcp_xyz:='0 0 0' tcp_rpy:='0 0 0' description_pkg:=openarm_description">
     <xacro:property name="ee_prefix" default=""/>
     <xacro:unless value="${arm_type == ''}">
@@ -39,7 +39,7 @@
         </geometry>
       </collision>
-      <xacro:if value="${gazebo}">
+      <!-- <xacro:if value="${gazebo}">
         <xacro:ee-inertials name="left_finger" />
-      </xacro:if>
+      </xacro:if> -->
     </link>
     <link name="${ee_prefix}right_finger">
@@ -56,7 +56,7 @@
         </geometry>
       </collision>
-      <xacro:if value="${gazebo}">
+      <!-- <xacro:if value="${gazebo}">
         <xacro:ee-inertials name="right_finger" />
-      </xacro:if>
+      </xacro:if> -->
     </link>
     <!-- <joint name="${ee_prefix}finger_joint1" type="prismatic">

File: openarm_description/urdf/ee/openarm_hand_arguments.xacro (robot description, xacro)
@@ -12,5 +12,5 @@
   <xacro:arg name="tcp_rpy" default="0 0 0" />
   <!-- Is the robot being simulated in gazebo? -->
-  <xacro:arg name="gazebo" default="false" />
+  <!-- <xacro:arg name="gazebo" default="false" /> -->
   <!-- Name of the description package -->
   <xacro:arg name="description_pkg" default="openarm_description" />

File: openarm_description/urdf/ee/openarm_hand_macro.xacro (robot description, xacro)
@@ -16,5 +16,5 @@
       </xacro:if>
   </xacro:macro>
-  <xacro:macro name="ee_link_with_sc" params="name prefix rpy:='0 0 0' gazebo:=false ee_kinematics_link">
+  <xacro:macro name="ee_link_with_sc" params="name prefix rpy:='0 0 0' ee_kinematics_link">
     <!-- sub-link defining detailed meshes for collision with environment -->
     <link name="${prefix}${name}">

File: openarm_description/urdf/robot/openarm_robot.xacro (robot description, xacro)
@@ -18,10 +18,8 @@
             hand:='false'
             ee_type:=''
-            gazebo:='false'
             ros2_control:=false
             can:=''
             use_fake_hardware:=false
             fake_sensor_commands:=false
-            gazebo_effort:=false
             no_prefix:='false'
             arm_prefix:=''
@@ -56,5 +54,4 @@
         xyz="${xyz}"
         rpy="${rpy}"
-        gazebo="${gazebo}"
         inertials="${body_inertials}"
         kinematics="${body_kinematics}"
@@ -69,5 +66,4 @@
         xyz="${left_arm_base_xyz}"
         rpy="${left_arm_base_rpy}"
-        gazebo="${gazebo}"
         joint_limits="${joint_limits}"
         inertials="${inertials}"
@@ -82,6 +78,4 @@
         use_fake_hardware="${use_fake_hardware}"
         fake_sensor_commands="${fake_sensor_commands}"
-        gazebo="${gazebo}"
-        gazebo_effort="${gazebo_effort}"
         hand="${hand}"
         bimanual="true"
@@ -97,5 +91,4 @@
         xyz="${right_arm_base_xyz}"
         rpy="${right_arm_base_rpy}"
-        gazebo="${gazebo}"
         joint_limits="${joint_limits}"
         inertials="${inertials}"
@@ -110,6 +103,4 @@
             use_fake_hardware="${use_fake_hardware}"
             fake_sensor_commands="${fake_sensor_commands}"
-            gazebo="${gazebo}"
-            gazebo_effort="${gazebo_effort}"
             hand="${hand}"
             bimanual="true"/>
@@ -127,5 +118,4 @@
                 tcp_xyz="$(arg tcp_xyz)"
                 tcp_rpy="$(arg tcp_rpy)"
-                gazebo="${gazebo}"
                 description_pkg="$(arg description_pkg)"
             />
@@ -141,5 +131,4 @@
                 tcp_xyz="$(arg tcp_xyz)"
                 tcp_rpy="$(arg tcp_rpy)"
-                gazebo="${gazebo}"
                 description_pkg="$(arg description_pkg)"
             />
@@ -153,5 +142,4 @@
         xyz="${xyz}"
         rpy="${rpy}"
-        gazebo="${gazebo}"
         joint_limits="${joint_limits}"
         kinematics="${kinematics}"
@@ -167,6 +155,4 @@
             use_fake_hardware="${use_fake_hardware}"
             fake_sensor_commands="${fake_sensor_commands}"
-            gazebo="${gazebo}"
-            gazebo_effort="${gazebo_effort}"
             hand="${hand}"
             bimanual="false"/>
@@ -188,5 +174,4 @@
             tcp_xyz="$(arg tcp_xyz)"
             tcp_rpy="$(arg tcp_rpy)"
-            gazebo="${gazebo}"
             description_pkg="$(arg description_pkg)"/>
         </xacro:if>

File: openarm_description/urdf/robot/v10.urdf.xacro (robot description, xacro)
@@ -17,6 +17,4 @@
     <xacro:property name="hand" value="false"/>
   </xacro:if>
-  <!-- Is the robot being simulated in gazebo?" -->
-  <xacro:arg name="gazebo" default="false" />
   <!-- If `gazebo` arg is set, to which frame shall $(arm_type)_link0 be parented. Empty string for not fixing at all -->
   <xacro:arg name="parent" default="world" />
@@ -34,5 +32,5 @@
   <xacro:arg name="fake_sensor_commands" default="false" />
   <!-- Should the robot be spawned in Gazebo with effort interfaces?" -->
-  <xacro:arg name="gazebo_effort" default="false" />
+  <!-- <xacro:arg name="gazebo_effort" default="false" /> -->
   <!-- For a multi arm setup, we need a threaded robot running async-->
   <xacro:arg name="bimanual" default="false" />
@@ -54,5 +52,4 @@
   body_kinematics_link="${xacro.load_yaml('$(find openarm_description)/config/body/v10/kinematics.yaml')}"
   ee_kinematics_link="${xacro.load_yaml('$(find openarm_description)/config/hand/openarm_hand/kinematics_link.yaml')}"
-  gazebo="$(arg gazebo)"
   hand="$(arg hand)"
   ee_type="$(arg ee_type)"
@@ -61,5 +58,4 @@
   use_fake_hardware="$(arg use_fake_hardware)"
   fake_sensor_commands="$(arg fake_sensor_commands)"
-  gazebo_effort="$(arg gazebo_effort)"
   no_prefix="$(arg no_prefix)"
   arm_prefix=""
