Commit message: fix: joint limits

File: openarm_description/urdf/ee/ee_with_one_link.xacro (robot description, xacro)
@@ -2,5 +2,5 @@
 <robot xmlns:xacro="http://www.ros.org/wiki/xacro" name="ee_with_one_link">
   <!-- safety_distance: Minimum safety distance in [m] by which the collision volumes are expanded and which is enforced during robot motions -->
-  <xacro:macro name="ee_with_one_link" params="connected_to:='' arm_type arm_prefix:='' ee_type ee_inertials rpy_ee:='0 0 0' xyz_ee:='0 0 0' tcp_xyz:='0 0 0' tcp_rpy:='0 0 0' gazebo:=false description_pkg:=openarm_description with_sc:=false">
+  <xacro:macro name="ee_with_one_link" params="connected_to:='' arm_type arm_prefix:='' ee_type ee_inertials rpy_ee:='0 0 0' xyz_ee:='0 0 0' tcp_xyz:='0 0 0' tcp_rpy:='0 0 0' description_pkg:=openarm_description with_sc:=false">
     <xacro:property name="ee_prefix" default="robot_"/>
     <xacro:unless value="${arm_type == ''}">
@@ -14,5 +14,5 @@
       </joint>
     </xacro:unless>
-    <xacro:ee_link_with_sc name="${ee_type}" gazebo="${gazebo}" />
+    <xacro:ee_link_with_sc name="${ee_type}"/>
     <!-- Define the ${ee_type}_tcp frame -->
     <link name="${ee_prefix}${ee_type}_tcp" />

File: openarm_description/urdf/ee/openarm_hand.xacro (robot description, xacro)
@@ -21,5 +21,4 @@
     <link name="${ee_prefix}hand_tcp" />
     <joint name="${ee_prefix}hand_tcp_joint" type="fixed">
-      <!-- <origin xyz="0 0.1 0.06" rpy="${tcp_rpy}" /> -->
       <origin xyz="${tcp_xyz}" rpy="${tcp_rpy}" />
       <parent link="${ee_prefix}hand" />

File: openarm_description/urdf/robot/openarm_robot.xacro (robot description, xacro)
@@ -191,5 +191,4 @@
             tcp_xyz="$(arg tcp_xyz)"
             tcp_rpy="$(arg tcp_rpy)"
-            gazebo="${gazebo}"
             description_pkg="$(arg description_pkg)"
         />
