Commit message: delete: gomi file

File: openarm_description/urdf/ee/openarm_hand.xacro (robot description, xacro)
@@ -2,5 +2,5 @@
 <robot xmlns:xacro="http://www.ros.org/wiki/xacro" name="hand">
   <!-- safety_distance: Minimum safety distance in [m] by which the collision volumes are expanded and which is enforced during robot motions -->
-  <xacro:macro name="openarm_hand" params="connected_to:='' arm_type arm_prefix:='' ee_type ee_inertials ee_kinematics_link rpy_ee:='0 0 0' xyz_ee:='0 0 0' tcp_xyz:='0 0 0.0' tcp_rpy:='0 0 0' gazebo:=false description_pkg:=openarm_description">
+  <xacro:macro name="openarm_hand" params="connected_to:='' arm_type arm_prefix:='' ee_type ee_inertials ee_kinematics_link rpy_ee:='0 0 0' xyz_ee:='0 0 0' tcp_xyz:='0 0.1 0' tcp_rpy:='0 0 0' gazebo:=false description_pkg:=openarm_description">
     <xacro:property name="ee_prefix" default=""/>
     <xacro:unless value="${arm_type == ''}">

File: openarm_description/urdf/robot/openarm_robot.xacro (robot description, xacro)
@@ -15,4 +15,8 @@
             xyz:='0 0 0'
             rpy:='0 0 0'
+            xyz_ee='0 0 0'
+            xyz_rpy='0 0 0'
+            tcp_xyz='0 0 0'
+            tcp_rpy='0 0 0'
             hand:='true'
             ee_type:=none

File: openarm_description/urdf/robot/v10.urdf.xacro (robot description, xacro)
@@ -64,4 +64,8 @@
   body_connected_to="world"
   bimanual="$(arg bimanual)"
+  xyz_ee='0 0 0'
+  xyz_rpy='0 0 0'
+  tcp_xyz='0 0 0'
+  tcp_rpy='0 0 0'
   right_arm_base_xyz="$(arg right_arm_base_xyz)"
   left_arm_base_xyz="$(arg left_arm_base_xyz)"

Commit message: fix: bimanual joint name

File: openarm_description/urdf/ee/openarm_hand.xacro (robot description, xacro)
@@ -10,5 +10,5 @@
     <xacro:unless value="${connected_to == ''}">
       <!-- <joint name="${ee_prefix}hand_joint" type="fixed"> -->
-      <joint name="openarm_hand_joint" type="fixed">
+      <joint name="${arm_prefix}openarm_hand_joint" type="fixed">
         <parent link="${connected_to}" />
         <child link="${ee_prefix}hand" />

File: openarm_description/urdf/robot/openarm_robot.xacro (robot description, xacro)
@@ -77,4 +77,5 @@
         kinematics_link="${kinematics_link}"
         kinematics_offset="${kinematics_offset}" />
+        <xacro:if value="${ros2_control}">
         <xacro:openarm_arm_ros2_control
         arm_type="${arm_type}"
@@ -87,5 +88,6 @@
         hand="${hand}"
         bimanual="true"
-      />
+        />
+       </xacro:if>
         <!-- right arm -->
         <xacro:openarm_arm
@@ -103,18 +105,19 @@
         kinematics_link="${kinematics_link}"
         kinematics_offset="${kinematics_offset}" />
-        <xacro:openarm_arm_ros2_control
-        arm_type="${arm_type}"
-        arm_prefix="right_"
-        can="can0"
-        use_fake_hardware="${use_fake_hardware}"
-        fake_sensor_commands="${fake_sensor_commands}"
-        gazebo="${gazebo}"
-        gazebo_effort="${gazebo_effort}"
-        hand="${hand}"
-        bimanual="true"
-        />
+        <xacro:if value="${ros2_control}">
+            <xacro:openarm_arm_ros2_control
+            arm_type="${arm_type}"
+            arm_prefix="right_"
+            can="can0"
+            use_fake_hardware="${use_fake_hardware}"
+            fake_sensor_commands="${fake_sensor_commands}"
+            gazebo="${gazebo}"
+            gazebo_effort="${gazebo_effort}"
+            hand="${hand}"
+            bimanual="true"/>
+        </xacro:if>
         <xacro:if value="${hand and ee_type == 'openarm_hand'}">
             <xacro:openarm_hand
-                connected_to="left_${arm_type}_link8"
+                connected_to="left_openarm_link8"
                 arm_type="${arm_type}"
                 arm_prefix="left_"
@@ -130,5 +133,5 @@
             />
             <xacro:openarm_hand
-                connected_to="right_${arm_type}_link8"
+                connected_to="right_openarm_link8"
                 arm_type="${arm_type}"
                 arm_prefix="right_"
@@ -159,4 +162,5 @@
         connected_to=""
         />
+        <xacro:if value="${ros2_control}">
         <xacro:openarm_arm_ros2_control
             arm_type="${arm_type}"
@@ -168,6 +172,6 @@
             gazebo_effort="${gazebo_effort}"
             hand="${hand}"
-            bimanual="false"
-        />
+            bimanual="false"/>
+        </xacro:if>
         <xacro:if value="${hand and ee_type == 'openarm_hand'}">
         <xacro:property name="special_connection" value="$(arg special_connection)" />
@@ -186,6 +190,5 @@
             tcp_rpy="$(arg tcp_rpy)"
             gazebo="${gazebo}"
-            description_pkg="$(arg description_pkg)"
-        />
+            description_pkg="$(arg description_pkg)"/>
         </xacro:if>
         <!-- <xacro:if value="${hand and ee_type != 'none' and ee_type != 'openarm_hand'}">

File: openarm_description/urdf/robot/v10.urdf (robot description, URDF)
Before this commit: robot openarm, 9 links, 8 joints
Links:
- removed link v10_link0
- removed link v10_link1
- removed link v10_link2
- removed link v10_link3
- removed link v10_link4
- removed link v10_link5
- removed link v10_link6
- removed link v10_link7
- removed link v10_link8
- added link openarm_hand
- added link openarm_hand_tcp
- added link openarm_left_finger; collision mesh filename=package://openarm_description/meshes/ee/openarm_hand/collis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 scale=0.001 0.001 0.001; visual mesh filename=package://openarm_description/meshes/ee/openarm_hand/visual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 scale=0.001 0.001 0.001
- added link openarm_link0, mass 1.1432284943239561; collision mesh filename=package://openarm_description/meshes/arm/v10/collision/link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 scale=0.001 -0.001 0.001; visual mesh filename=package://openarm_description/meshes/arm/v10/visual/link0.d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 scale=0.001 -0.001 0.001
- added link openarm_link1, mass 1.1416684646202298; collision mesh filename=package://openarm_description/meshes/arm/v10/collision/link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 scale=0.001 -0.001 0.001; visual mesh filename=package://openarm_description/meshes/arm/v10/visual/link1.d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 scale=0.001 -0.001 0.001
- added link openarm_link2, mass 0.2775092746011571; collision mesh filename=package://openarm_description/meshes/arm/v10/collision/link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 scale=0.001 -0.001 0.001; visual mesh filename=package://openarm_description/meshes/arm/v10/visual/link2.d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 scale=0.001 -0.001 0.001
- added link openarm_link3, mass 1.073863338202347; collision mesh filename=package://openarm_description/meshes/arm/v10/collision/link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 scale=0.001 -0.001 0.001; visual mesh filename=package://openarm_description/meshes/arm/v10/visual/link3.d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 scale=0.001 -0.001 0.001
- added link openarm_link4, mass 1.3699337287025453; collision mesh filename=package://openarm_description/meshes/arm/v10/collision/link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 scale=0.001 0.001 0.001; visual mesh filename=package://openarm_description/meshes/arm/v10/visual/link4.d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 scale=0.001 0.001 0.001
- added link openarm_link5, mass 0.5506588026168502; collision mesh filename=package://openarm_description/meshes/arm/v10/collision/link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 scale=0.001 -0.001 0.001; visual mesh filename=package://openarm_description/meshes/arm/v10/visual/link5.d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 scale=0.001 -0.001 0.001
- added link openarm_link6, mass 0.3540202773187987; collision mesh filename=package://openarm_description/meshes/arm/v10/collision/link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 scale=0.001 -0.001 0.001; visual mesh filename=package://openarm_description/meshes/arm/v10/visual/link6.d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 scale=0.001 -0.001 0.001
- added link openarm_link7, mass 0.5499771327380578; collision mesh filename=package://openarm_description/meshes/arm/v10/collision/link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 scale=0.001 -0.001 0.001; visual mesh filename=package://openarm_description/meshes/arm/v10/visual/link7.d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 scale=0.001 -0.001 0.001
- added link openarm_link8
- added link openarm_right_finger; collision mesh filename=package://openarm_description/meshes/ee/openarm_hand/collis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 scale=0.001 -0.001 0.001; visual mesh filename=package://openarm_description/meshes/ee/openarm_hand/visual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 scale=0.001 -0.001 0.001
Joints:
- removed joint v10_joint1
- removed joint v10_joint2
- removed joint v10_joint3
- removed joint v10_joint4
- removed joint v10_joint5
- removed joint v10_joint6
- removed joint v10_joint7
- removed joint v10_joint8
- added joint openarm_finger_joint1: type prismatic, parent openarm_hand, child openarm_right_finger, origin xyz=0 0.095 0 rpy=0 0 0, axis 0 -1 0, limit lower=0.0 upper=0.044 effort=100 velocity=0.2
- added joint openarm_finger_joint2: type prismatic, parent openarm_hand, child openarm_left_finger, origin xyz=0 0.105 0 rpy=0 0 0, axis 0 1 0, limit lower=0.0 upper=0.044 effort=100 velocity=0.2, mimic joint=openarm_finger_joint1
- added joint openarm_hand_joint: type fixed, parent openarm_link8, child openarm_hand, origin xyz=0 0 0 rpy=0 0 0
- added joint openarm_hand_tcp_joint: type fixed, parent openarm_hand, child openarm_hand_tcp, origin xyz=0 0 0.0 rpy=0 0 0
- added joint openarm_joint1: type revolute, parent openarm_link0, child openarm_link1, origin xyz=0.0 0.0 0.0625 rpy=0 0 0, axis 0 0 1, limit lower=-1.396263 upper=3.490659 effort=100 velocity=100
- added joint openarm_joint2: type revolute, parent openarm_link1, child openarm_link2, origin xyz=-0.0301 0.0 0.06 rpy=0 0 0, axis -1 0 0, limit lower=-1.745329 upper=1.745329 effort=100 velocity=100
- added joint openarm_joint3: type revolute, parent openarm_link2, child openarm_link3, origin xyz=0.0301 0.0 0.06625 rpy=0 0 0, axis 0 0 1, limit lower=-1.570796 upper=1.570796 effort=100 velocity=100
- added joint openarm_joint4: type revolute, parent openarm_link3, child openarm_link4, origin xyz=-0.0 0.0315 0.15375 rpy=0 0 0, axis 0 1 0, limit lower=0.0 upper=2.443461 effort=100 velocity=100
- added joint openarm_joint5: type revolute, parent openarm_link4, child openarm_link5, origin xyz=0.0 -0.0315 0.0955 rpy=0 0 0, axis 0 0 1, limit lower=-1.570796 upper=1.570796 effort=100 velocity=100
- added joint openarm_joint6: type revolute, parent openarm_link5, child openarm_link6, origin xyz=0.0375 0.0 0.1205 rpy=0 0 0, axis 1 0 0, limit lower=-0.785398 upper=0.785398 effort=100 velocity=100
- added joint openarm_joint7: type revolute, parent openarm_link6, child openarm_link7, origin xyz=-0.0375 0.0 0.0 rpy=0 0 0, axis 0 1 0, limit lower=-1.570796 upper=1.570796 effort=100 velocity=100
- added joint openarm_joint8: type fixed, parent openarm_link7, child openarm_link8, origin xyz=1e-06 -0.098 0.114501 rpy=0 0 0

Commit message: fix: ee_type none error

File: openarm_description/urdf/ee/openarm_hand.xacro (robot description, xacro)
@@ -21,6 +21,6 @@
     <link name="${ee_prefix}hand_tcp" />
     <joint name="${ee_prefix}hand_tcp_joint" type="fixed">
-      <origin xyz="0 0.1 0.06" rpy="${tcp_rpy}" />
-      <!-- <origin xyz="${tcp_xyz}" rpy="${tcp_rpy}" /> -->
+      <!-- <origin xyz="0 0.1 0.06" rpy="${tcp_rpy}" /> -->
+      <origin xyz="${tcp_xyz}" rpy="${tcp_rpy}" />
       <parent link="${ee_prefix}hand" />
       <child link="${ee_prefix}hand_tcp" />

File: openarm_description/urdf/ee/openarm_hand_arguments.xacro (robot description, xacro)
@@ -1,16 +1,12 @@
 <?xml version="1.0" encoding="utf-8"?>
 <robot xmlns:xacro="http://www.ros.org/wiki/xacro">
-  <!-- Name for the robot -->
-  <xacro:arg name="arm_type" default="v10" />
-  <!-- End-effector id" -->
-  <xacro:arg name="ee_type" default="openarm_hand" />
   <!-- Where is the end-effector connected to, if different from the robot flange?  -->
   <xacro:arg name="special_connection" default="" />
   <!-- Position offset between ee and parent frame -->
-  <xacro:arg name="xyz_ee" default="0 0 0" />
+  <xacro:arg name="xyz_ee" default="0 0 0.0" />
   <!-- Rotation offset between ee and parent frame -->
   <xacro:arg name="rpy_ee" default= "0 0 0" />
   <!-- Position offset between ee frame and tcp frame -->
-  <xacro:arg name="tcp_xyz" default="0 0 0.0" />
+  <xacro:arg name="tcp_xyz" default="0 0.0 0.0" />
   <!-- Rotation offset between ee frame and tcp frame -->
   <xacro:arg name="tcp_rpy" default="0 0 0" />

File: openarm_description/urdf/ee/openarm_hand_macro.xacro (robot description, xacro)
@@ -26,4 +26,5 @@
       </visual>
       <collision name="${prefix}${name}_collision">
+        <xacro:openarm-ee-kinematics-link config="${ee_kinematics_link}" name="${name}" />
         <geometry>
           <mesh filename="package://openarm_description/meshes/ee/${ee_type}/collision/${name}.stl" scale="0.001 0.001 0.001" />

File: openarm_description/urdf/robot/openarm_robot.xacro (robot description, xacro)
@@ -16,10 +16,6 @@
             xyz:='0 0 0'
             rpy:='0 0 0'
-            xyz_ee='0 0 0'
-            xyz_rpy='0 0 0'
-            tcp_xyz='0 0 0'
-            tcp_rpy='0 0 0'
-            hand:='true'
-            ee_type:=none
+            hand:='false'
+            ee_type:=''
             gazebo:='false'
             ros2_control:=false
@@ -33,5 +29,5 @@
             arm_connected_to='base'
             body_connected_to='world'
-            bimanual:=true
+            bimanual:=false
             right_arm_base_xyz='0 0 0'
             left_arm_base_xyz='0 0 0'
@@ -45,6 +41,8 @@
     <xacro:include filename="$(find openarm_description)/urdf/ee/openarm_hand.xacro" />
     <xacro:include filename="$(find openarm_description)/urdf/ee/openarm_hand_macro.xacro" />
-    <xacro:include filename="$(find openarm_description)/urdf/ee/${ee_type}_arguments.xacro" />
     <xacro:include filename="$(find openarm_description)/urdf/ros2_control/openarm.ros2_control.xacro" />
+    <xacro:if value="${ee_type != 'none'}">
+        <xacro:include filename="$(find openarm_description)/urdf/ee/${ee_type}_arguments.xacro" />
+      </xacro:if>
     <xacro:property name="arm_prefix_modified" value="${'' if arm_prefix == '' else arm_prefix + '_'}" />
     <xacro:property name="body_prefix_modified" value="${'' if body_prefix == '' else body_prefix + '_'}" />
@@ -117,5 +115,5 @@
             bimanual="true"/>
         </xacro:if>
-        <xacro:if value="${hand and ee_type == 'openarm_hand'}">
+        <xacro:if value="$(eval hand and ee_type == 'openarm_hand')">
             <xacro:openarm_hand
                 connected_to="openarm_left_link8"
@@ -178,4 +176,5 @@
         <!-- <xacro:property name="connection" value="${special_connection if special_connection != '' else arm_type + '_link8'}" /> -->
         <xacro:property name="connection" value="${special_connection if special_connection != '' else 'openarm' + '_link8'}" />
+        <xacro:if value="$(eval hand and ee_type == 'openarm_hand')">
         <xacro:openarm_hand
             connected_to="${arm_prefix_modified}${connection}"
@@ -191,4 +190,5 @@
             gazebo="${gazebo}"
             description_pkg="$(arg description_pkg)"/>
+        </xacro:if>
         </xacro:if>
         <!-- <xacro:if value="${hand and ee_type != 'none' and ee_type != 'openarm_hand'}">

File: openarm_description/urdf/robot/v10.urdf.xacro (robot description, xacro)
@@ -14,4 +14,7 @@
   <!-- Should an end-effector be mounted at the flange?" -->
   <xacro:arg name="hand" default="true" />
+  <xacro:if value="$(eval ee_type == 'none')">
+    <xacro:property name="hand" value="false"/>
+  </xacro:if>
   <!-- Is the robot being simulated in gazebo?" -->
   <xacro:arg name="gazebo" default="false" />
@@ -65,8 +68,4 @@
   body_connected_to="world"
   bimanual="$(arg bimanual)"
-  xyz_ee='0 0 0'
-  xyz_rpy='0 0 0'
-  tcp_xyz='0 0.1 0.06'
-  tcp_rpy='0 0 0'
   right_arm_base_xyz="$(arg right_arm_base_xyz)"
   left_arm_base_xyz="$(arg left_arm_base_xyz)"

Commit message: fix: finger force limit

File: openarm_description/urdf/ee/openarm_hand.xacro (robot description, xacro)
@@ -79,5 +79,5 @@
       <origin xyz="0 0.095 0" rpy="0 0 0" />
       <axis xyz="0 -1 0" />
-      <limit effort="100" lower="0.0" upper="0.044" velocity="0.2" />
+      <limit effort="10" lower="0.0" upper="0.044" velocity="0.2" />
     </joint>
     <joint name="${ee_prefix}finger_joint2" type="prismatic">
@@ -86,5 +86,5 @@
       <origin xyz="0 0.105 0" rpy="0 0 0" />
       <axis xyz="0 1 0" />
-      <limit effort="100" lower="0.0" upper="0.044" velocity="0.2" />
+      <limit effort="10" lower="0.0" upper="0.044" velocity="0.2" />
       <mimic joint="${ee_prefix}finger_joint1" />
     </joint>

File: openarm_description/urdf/robot/openarm_robot.xacro (robot description, xacro)
@@ -42,5 +42,5 @@
     <xacro:if value="${ee_type != 'none'}">
         <xacro:include filename="$(find openarm_description)/urdf/ee/${ee_type}_arguments.xacro" />
-      </xacro:if>
+    </xacro:if>
     <xacro:property name="arm_prefix_modified" value="${'' if arm_prefix == '' else arm_prefix + '_'}" />
     <xacro:property name="body_prefix_modified" value="${'' if body_prefix == '' else body_prefix + '_'}" />

Commit message: delete: gazebo setting

File: openarm_description/urdf/ee/openarm_hand.xacro (robot description, xacro)
@@ -16,5 +16,5 @@
       </joint>
     </xacro:unless>
-    <!-- <xacro:ee_link_with_sc name="hand" gazebo="${gazebo}" prefix="${ee_prefix}" ee_kinematics_link="${ee_kinematics_link}"/> -->
+    <!-- <xacro:ee_link_with_sc name="hand" prefix="${ee_prefix}" ee_kinematics_link="${ee_kinematics_link}"/> -->
     <link name="${ee_prefix}hand"/>
     <!-- Define the hand_tcp frame -->
@@ -38,7 +38,4 @@
         </geometry>
       </collision>
-      <!-- <xacro:if value="${gazebo}">
-        <xacro:ee-inertials name="left_finger" />
-      </xacro:if> -->
     </link>
     <link name="${ee_prefix}right_finger">
@@ -55,7 +52,4 @@
         </geometry>
       </collision>
-      <!-- <xacro:if value="${gazebo}">
-        <xacro:ee-inertials name="right_finger" />
-      </xacro:if> -->
     </link>
     <!-- <joint name="${ee_prefix}finger_joint1" type="prismatic">
@@ -79,5 +73,5 @@
       <origin xyz="0 0.095 0" rpy="0 0 0" />
       <axis xyz="0 -1 0" />
-      <limit effort="10" lower="0.0" upper="0.044" velocity="0.2" />
+      <limit effort="10" lower="0.0" upper="0.044" velocity="1.0" />
     </joint>
     <joint name="${ee_prefix}finger_joint2" type="prismatic">
@@ -86,5 +80,5 @@
       <origin xyz="0 0.105 0" rpy="0 0 0" />
       <axis xyz="0 1 0" />
-      <limit effort="10" lower="0.0" upper="0.044" velocity="0.2" />
+      <limit effort="10" lower="0.0" upper="0.044" velocity="1.0" />
       <mimic joint="${ee_prefix}finger_joint1" />
     </joint>

Commit message: fix: hand inertia

File: openarm_description/urdf/ee/openarm_hand.xacro (robot description, xacro)
@@ -8,4 +8,6 @@
       <xacro:property name="ee_prefix" value="openarm_${arm_prefix}" />
     </xacro:unless>
+    <xacro:ee_link_with_sc name="hand" prefix="${ee_prefix}" ee_kinematics_link="${ee_kinematics_link}"/>
+    <!-- <link name="${ee_prefix}hand"/> -->
     <xacro:unless value="${connected_to == ''}">
       <!-- <joint name="${ee_prefix}hand_joint" type="fixed"> -->
@@ -16,6 +18,4 @@
       </joint>
     </xacro:unless>
-    <!-- <xacro:ee_link_with_sc name="hand" prefix="${ee_prefix}" ee_kinematics_link="${ee_kinematics_link}"/> -->
-    <link name="${ee_prefix}hand"/>
     <!-- Define the hand_tcp frame -->
     <link name="${ee_prefix}hand_tcp" />
@@ -38,4 +38,5 @@
         </geometry>
       </collision>
+      <xacro:ee-inertials name="left_finger"/>
     </link>
     <link name="${ee_prefix}right_finger">
@@ -52,24 +53,10 @@
         </geometry>
       </collision>
+      <xacro:ee-inertials name="right_finger"/>
     </link>
-    <!-- <joint name="${ee_prefix}finger_joint1" type="prismatic">
-      <parent link="${ee_prefix}hand" />
-      <child link="${ee_prefix}right_finger" />
-      <origin xyz="0 0.05 0" rpy="0 0 0" />
-      <axis xyz="0 -1 0" />
-      <limit effort="100" lower="0.0" upper="0.044" velocity="0.2" />
-    </joint>
-    <joint name="${ee_prefix}finger_joint2" type="prismatic">
-      <parent link="${ee_prefix}hand" />
-      <child link="${ee_prefix}left_finger" />
-      <origin xyz="0 0.15 0" rpy="0 0 0" />
-      <axis xyz="0 1 0" />
-      <limit effort="100" lower="0.0" upper="0.044" velocity="0.2" />
-      <mimic joint="${ee_prefix}finger_joint1" />
-    </joint> -->
     <joint name="${ee_prefix}finger_joint1" type="prismatic">
       <parent link="${ee_prefix}hand" />
       <child link="${ee_prefix}right_finger" />
-      <origin xyz="0 0.095 0" rpy="0 0 0" />
+      <origin xyz="0 -0.026 0.115" rpy="0 0 0" />
       <axis xyz="0 -1 0" />
       <limit effort="10" lower="0.0" upper="0.044" velocity="1.0" />
@@ -78,5 +65,5 @@
       <parent link="${ee_prefix}hand" />
       <child link="${ee_prefix}left_finger" />
-      <origin xyz="0 0.105 0" rpy="0 0 0" />
+      <origin xyz="0 -0.016 0.115" rpy="0 0 0" />
       <axis xyz="0 1 0" />
       <limit effort="10" lower="0.0" upper="0.044" velocity="1.0" />
