Commit message: add v20 support

File: openarm_bimanual_moveit_config/config/v10/openarm_bimanual.urdf.xacro (robot description, xacro)
@@ -15,6 +15,5 @@
     <xacro:arg name="initial_positions_file" default="initial_positions.yaml" />
     <xacro:arg name="hardware_type" default="real" />
-    <!-- Import openarm_bimanual urdf file -->
-    <xacro:include filename="$(find openarm_description)/urdf/robot/v10.urdf.xacro" />
+    <xacro:include filename="$(find openarm_description)/urdf/robot/v10/v10.urdf.xacro" />
     <link name="base_link"/>
     <joint name="world_to_pedestal" type="fixed">

File: openarm_bimanual_moveit_config/config/v20/openarm_bimanual.urdf.xacro (robot description, xacro)
@@ -1,2 +1,3 @@
+<?xml version="1.0"?>
 <!--
 　Copyright 2025 Enactic, Inc.
@@ -11,11 +12,13 @@
 　limitations under the License.
 -->
-<library path="openarm_hardware">
-  <class name="openarm_hardware/OpenArmHW"
-         type="openarm_hardware::OpenArmHW"
-         base_class_type="hardware_interface::SystemInterface">
-    <description>
-      ros2_control hardware interface for OpenArm .
-    </description>
-  </class>
-</library>
+<robot xmlns:xacro="http://www.ros.org/wiki/xacro" name="openarm_bimanual">
+    <xacro:arg name="initial_positions_file" default="initial_positions.yaml" />
+    <xacro:arg name="hardware_type" default="real" />
+    <xacro:include filename="$(find openarm_description)/urdf/robot/v20/v20.urdf.xacro" />
+    <link name="base_link"/>
+    <joint name="world_to_pedestal" type="fixed">
+        <parent link="world"/>
+        <child link="base_link"/>
+        <origin xyz="0.0 0.0 0.0" rpy="0.0 0.0 0.0"/>
+    </joint>
+</robot>
